File: Hardware/MADC_ARTY/AutoZero.kicad_sch (KiCad schematic)
At the start: 13 parts, among them U12 ADG419BRM, U13 ADG419BRM

Commit message: PCB and schematic
Changed lines of the file:
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@@
 		(dnp no)
 		(fields_autoplaced yes)
-		(property "Reference" "#PWR081"
+		(property "Reference" "#PWR81"
 			(at 146.05 87.63 0)
 			(effects
@@
 			(project "MADC_ARTY"
 				(path "/eadab778-ea7c-433e-b0bd-0d0c238907e0/37dfacfc-f3f5-4a09-9e7e-ab0b8ea302f6/0c7976b3-7b09-4b41-8942-e28e3585795d"
-					(reference "#PWR0120")
-					(unit 1)
-				)
-				(path "/eadab778-ea7c-433e-b0bd-0d0c238907e0/37dfacfc-f3f5-4a09-9e7e-ab0b8ea302f6/e5f31b97-6641-44bd-9522-ccfcbaab9fbc"
-					(reference "#PWR081")
+					(reference "#PWR120")
+					(unit 1)
+				)
+				(path "/eadab778-ea7c-433e-b0bd-0d0c238907e0/37dfacfc-f3f5-4a09-9e7e-ab0b8ea302f6/e5f31b97-6641-44bd-9522-ccfcbaab9fbc"
+					(reference "#PWR81")
 					(unit 1)
 				)
@@
 		(dnp no)
 		(fields_autoplaced yes)
-		(property "Reference" "#PWR080"
+		(property "Reference" "#PWR80"
 			(at 127 195.58 0)
 			(effects
@@
 			(project "MADC_ARTY"
 				(path "/eadab778-ea7c-433e-b0bd-0d0c238907e0/37dfacfc-f3f5-4a09-9e7e-ab0b8ea302f6/0c7976b3-7b09-4b41-8942-e28e3585795d"
-					(reference "#PWR0119")
-					(unit 1)
-				)
-				(path "/eadab778-ea7c-433e-b0bd-0d0c238907e0/37dfacfc-f3f5-4a09-9e7e-ab0b8ea302f6/e5f31b97-6641-44bd-9522-ccfcbaab9fbc"
-					(reference "#PWR080")
+					(reference "#PWR119")
+					(unit 1)
+				)
+				(path "/eadab778-ea7c-433e-b0bd-0d0c238907e0/37dfacfc-f3f5-4a09-9e7e-ab0b8ea302f6/e5f31b97-6641-44bd-9522-ccfcbaab9fbc"
+					(reference "#PWR80")
 					(unit 1)
 				)
@@
 		(on_board yes)
 		(dnp no)
-		(property "Reference" "#PWR074"
+		(property "Reference" "#PWR74"
 			(at 101.6 195.58 0)
 			(effects
@@
 		)
 		(property "Value" "GND"
-			(at 101.6 194.31 0)
+			(at 101.6 193.04 0)
 			(effects
 				(font
@@
 			(project "MADC_ARTY"
 				(path "/eadab778-ea7c-433e-b0bd-0d0c238907e0/37dfacfc-f3f5-4a09-9e7e-ab0b8ea302f6/0c7976b3-7b09-4b41-8942-e28e3585795d"
-					(reference "#PWR0113")
-					(unit 1)
-				)
-				(path "/eadab778-ea7c-433e-b0bd-0d0c238907e0/37dfacfc-f3f5-4a09-9e7e-ab0b8ea302f6/e5f31b97-6641-44bd-9522-ccfcbaab9fbc"
-					(reference "#PWR074")
+					(reference "#PWR113")
+					(unit 1)
+				)
+				(path "/eadab778-ea7c-433e-b0bd-0d0c238907e0/37dfacfc-f3f5-4a09-9e7e-ab0b8ea302f6/e5f31b97-6641-44bd-9522-ccfcbaab9fbc"
+					(reference "#PWR74")
 					(unit 1)
 				)
@@
 		(dnp no)
 		(fields_autoplaced yes)
-		(property "Reference" "#PWR066"
+		(property "Reference" "#PWR66"
 			(at 17.78 186.69 0)
 			(effects
@@
 			(project "MADC_ARTY"
 				(path "/eadab778-ea7c-433e-b0bd-0d0c238907e0/37dfacfc-f3f5-4a09-9e7e-ab0b8ea302f6/0c7976b3-7b09-4b41-8942-e28e3585795d"
-					(reference "#PWR0105")
-					(unit 1)
-				)
-				(path "/eadab778-ea7c-433e-b0bd-0d0c238907e0/37dfacfc-f3f5-4a09-9e7e-ab0b8ea302f6/e5f31b97-6641-44bd-9522-ccfcbaab9fbc"
-					(reference "#PWR066")
+					(reference "#PWR105")
+					(unit 1)
+				)
+				(path "/eadab778-ea7c-433e-b0bd-0d0c238907e0/37dfacfc-f3f5-4a09-9e7e-ab0b8ea302f6/e5f31b97-6641-44bd-9522-ccfcbaab9fbc"
+					(reference "#PWR66")
 					(unit 1)
 				)
@@
 		(dnp no)
 		(fields_autoplaced yes)
-		(property "Reference" "#PWR068"
+		(property "Reference" "#PWR68"
 			(at 41.91 186.69 0)
 			(effects
@@
 			(project "MADC_ARTY"
 				(path "/eadab778-ea7c-433e-b0bd-0d0c238907e0/37dfacfc-f3f5-4a09-9e7e-ab0b8ea302f6/0c7976b3-7b09-4b41-8942-e28e3585795d"
-					(reference "#PWR0107")
-					(unit 1)
-				)
-				(path "/eadab778-ea7c-433e-b0bd-0d0c238907e0/37dfacfc-f3f5-4a09-9e7e-ab0b8ea302f6/e5f31b97-6641-44bd-9522-ccfcbaab9fbc"
-					(reference "#PWR068")
+					(reference "#PWR107")
+					(unit 1)
+				)
+				(path "/eadab778-ea7c-433e-b0bd-0d0c238907e0/37dfacfc-f3f5-4a09-9e7e-ab0b8ea302f6/e5f31b97-6641-44bd-9522-ccfcbaab9fbc"
+					(reference "#PWR68")
 					(unit 1)
 				)
@@
 		(dnp no)
 		(fields_autoplaced yes)
-		(property "Reference" "#PWR078"
+		(property "Reference" "#PWR78"
 			(at 120.65 95.25 0)
 			(effects
@@
 			(project "MADC_ARTY"
 				(path "/eadab778-ea7c-433e-b0bd-0d0c238907e0/37dfacfc-f3f5-4a09-9e7e-ab0b8ea302f6/0c7976b3-7b09-4b41-8942-e28e3585795d"
-					(reference "#PWR0117")
-					(unit 1)
-				)
-				(path "/eadab778-ea7c-433e-b0bd-0d0c238907e0/37dfacfc-f3f5-4a09-9e7e-ab0b8ea302f6/e5f31b97-6641-44bd-9522-ccfcbaab9fbc"
-					(reference "#PWR078")
+					(reference "#PWR117")
+					(unit 1)
+				)
+				(path "/eadab778-ea7c-433e-b0bd-0d0c238907e0/37dfacfc-f3f5-4a09-9e7e-ab0b8ea302f6/e5f31b97-6641-44bd-9522-ccfcbaab9fbc"
+					(reference "#PWR78")
 					(unit 1)
 				)
@@
 		(dnp no)
 		(fields_autoplaced yes)
-		(property "Reference" "#PWR070"
+		(property "Reference" "#PWR70"
 			(at 66.04 186.69 0)
 			(effects
@@
 			(project "MADC_ARTY"
 				(path "/eadab778-ea7c-433e-b0bd-0d0c238907e0/37dfacfc-f3f5-4a09-9e7e-ab0b8ea302f6/0c7976b3-7b09-4b41-8942-e28e3585795d"
-					(reference "#PWR0109")
-					(unit 1)
-				)
-				(path "/eadab778-ea7c-433e-b0bd-0d0c238907e0/37dfacfc-f3f5-4a09-9e7e-ab0b8ea302f6/e5f31b97-6641-44bd-9522-ccfcbaab9fbc"
-					(reference "#PWR070")
+					(reference "#PWR109")
+					(unit 1)
+				)
+				(path "/eadab778-ea7c-433e-b0bd-0d0c238907e0/37dfacfc-f3f5-4a09-9e7e-ab0b8ea302f6/e5f31b97-6641-44bd-9522-ccfcbaab9fbc"
+					(reference "#PWR70")
 					(unit 1)
 				)
@@
 		(dnp no)
 		(fields_autoplaced yes)
-		(property "Reference" "#PWR075"
+		(property "Reference" "#PWR75"
 			(at 107.95 85.09 0)
 			(effects
@@
 			(project "MADC_ARTY"
 				(path "/eadab778-ea7c-433e-b0bd-0d0c238907e0/37dfacfc-f3f5-4a09-9e7e-ab0b8ea302f6/0c7976b3-7b09-4b41-8942-e28e3585795d"
-					(reference "#PWR0114")
-					(unit 1)
-				)
-				(path "/eadab778-ea7c-433e-b0bd-0d0c238907e0/37dfacfc-f3f5-4a09-9e7e-ab0b8ea302f6/e5f31b97-6641-44bd-9522-ccfcbaab9fbc"
-					(reference "#PWR075")
-					(unit 1)
-				)
+					(reference "#PWR114")
+					(unit 1)
+				)
+				(path "/eadab778-ea7c-433e-b0bd-0d0c238907e0/37dfacfc-f3f5-4a09-9e7e-ab0b8ea302f6/e5f31b97-6641-44bd-9522-ccfcbaab9fbc"
+					(reference "#PWR75")
+					(unit 1)
+				)

Commit message: BOM
Parts:
- renumbered C27 to C29, C28 to C30, C29 to C31, C30 to C32, C31 to C33, C32 to C34, R39 to R45, R40 to R46, R41 to R47, R42 to R48, R43 to R49, U12 to U13, U13 to U14
