File: Hardware/MADC_ARTY/BlockDiagram.kicad_sch (KiCad schematic)
At the start: 2 parts, among them J1 Conn_01x01, J2 Conn_01x01

Commit message: Schematic
Other:
- added sheet ADC (ADC.kicad_sch)
- sheet Auto Zero ports: added AZ1_CTR, AZ2_CTR; removed AUTO_ZERO_CTR, INPUT_CTR
Changed lines of the file:
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@@
+	)
+	(sheet
+		(at 198.12 55.88)
+		(size 46.99 30.48)
+		(exclude_from_sim no)
+		(in_bom yes)
+		(on_board yes)
+		(dnp no)
+		(fields_autoplaced yes)
+		(stroke
+			(width 0.1524)
+			(type solid)
+		)
+		(fill
+			(color 0 0 0 0.0000)
+		)
+		(property "Sheetname" "ADC"
+			(at 198.12 55.1684 0)
+			(effects
+				(font
+					(size 1.27 1.27)
+				)
+				(justify left bottom)
+			)
+		)
+		(property "Sheetfile" "ADC.kicad_sch"
+			(at 198.12 86.9446 0)
+			(effects
+				(font
+					(size 1.27 1.27)
+				)
+				(justify left top)
+			)
+		)
+		(instances
+			(project "MADC_ARTY"
+				(path "/eadab778-ea7c-433e-b0bd-0d0c238907e0/37dfacfc-f3f5-4a09-9e7e-ab0b8ea302f6"
+					(page "7")
+				)
+			)
+		)
 	)
 	(sheet
@@
 			)
 		)
-		(pin "INPUT_CTR" input
-			(at 107.95 82.55 0)
-			(effects
-				(font
-					(size 1.27 1.27)
-				)
-				(justify right)
-			)
-		)
 		(pin "AIN_P" input
 			(at 76.2 59.69 180)
@@
 			)
 		)
-		(pin "AUTO_ZERO_CTR" input
-			(at 107.95 78.74 0)
-			(effects
-				(font
-					(size 1.27 1.27)
-				)
-				(justify right)
-			)
-		)
 		(pin "AZ_OUT_P" output
 			(at 107.95 59.69 0)
@@
 			(effects
 				(font
+					(size 1.27 1.27)
+				)
+				(justify right)
+			)
+		)
+		(pin "AZ2_CTR" input
+			(at 107.95 82.55 0)
+			(effects
+				(font
+					(size 1.27 1.27)
+				)
+				(justify right)
+			)
+		)
+		(pin "AZ1_CTR" input
+			(at 107.95 78.74 0)
+			(effects
+				(font

Commit message: Schematic
Other:
- added sheet PMOD (PMOD.kicad_sch)
- added sheet Voltage Reference (VoltageReference.kicad_sch)
- sheet ADC ports: added ADIN, AD_COMP, FGPA_AD_ID, FGPA_AD_IIN, FGPA_AD_IRN, FGPA_AD_IRP, FPGA_SW_VRH; removed none

Commit message: Schematic
Parts:
- J1, J2: footprint (none) -> MADC:S16N-PC
Other:
- sheet PMOD ports: added AD_COMP, AZ1_CTR, AZ2_CTR, FGPA_AD_ID, FGPA_AD_IIN, FGPA_AD_IRN, FGPA_AD_IRP, FPGA_SW_VRH, GAIN_x10, GAIN_x100; removed none
- moved on the sheet: J1, J2

Commit message: Schematic
Other:
- sheet Auto Zero ports: added AZ_CTR; removed AZ1_CTR, AZ2_CTR
- sheet PMOD ports: added none; removed AZ1_CTR, AZ2_CTR
Changed lines of the file:
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@@
-	(wire
-		(pts
-			(xy 93.98 74.93) (xy 128.27 74.93)
-		)
-		(stroke
-			(width 0)
-			(type default)
-		)
-	)
 	(wire
 		(pts
@@
 	(wire
 		(pts
-			(xy 128.27 85.09) (xy 214.63 85.09)
-		)
-		(stroke
-			(width 0)
-			(type default)
-		)
-	)
-	(wire
-		(pts
 			(xy 207.01 62.23) (xy 214.63 62.23)
 		)
@@
 		(pts
 			(xy 207.01 54.61) (xy 214.63 54.61)
-		)
-		(stroke
-			(width 0)
-			(type default)
-		)
-	)
-	(wire
-		(pts
-			(xy 128.27 74.93) (xy 128.27 85.09)
 		)
 		(stroke
@@
 			)
 		)
-		(pin "AZ2_CTR" output
-			(at 214.63 85.09 180)
-			(effects
-				(font
-					(size 1.27 1.27)
-				)
-				(justify left)
-			)
-		)
-		(pin "AZ1_CTR" output
-			(at 214.63 82.55 180)
-			(effects
-				(font
-					(size 1.27 1.27)
-				)
-				(justify left)
-			)
-		)
 		(pin "FGPA_AD_ID" output
 			(at 214.63 54.61 180)
@@
 			)
 		)
-		(pin "AZ2_CTR" input
-			(at 93.98 74.93 0)
-			(effects
-				(font
-					(size 1.27 1.27)
-				)
-				(justify right)
-			)
-		)
-		(pin "AZ1_CTR" input
+		(pin "AZ_CTR" input
 			(at 93.98 72.39 0)
 			(effects

Commit message: PCB and Schematic
Connections:
- net Auto Zero/AIN_N renamed Auto Zero1/AIN
- net Auto Zero/AIN_P renamed Auto Zero/AIN
Other:
- added sheet Analog Channels1 (AnalogChannels.kicad_sch)
- added sheet Auto Zero1 (AutoZero.kicad_sch)
- sheet Analog Channels ports: added IN, OUT; removed IN_N, IN_P, OUT_N, OUT_P
- sheet Auto Zero ports: added AIN, AZ_OUT; removed AIN_N, AIN_P, AZ_OUT_N, AZ_OUT_P
- sheet PMOD ports: added AZ_CTR; removed none
- moved on the sheet: J2

Commit message: PCB
Parts:
- added H1, H2, H3, H4: MountingHole, MountingHole:MountingHole_3.2mm_M3_DIN965_Pad, symbol Mechanical:MountingHole

Commit message: PCB and schematic
Other:
- sheet ADC ports: added AD_CMP, AD_ID, AD_IIN, AD_IN, AD_IRN, AD_IRP, SW_VRH; removed ADIN, AD_COMP, FGPA_AD_ID, FGPA_AD_IIN, FGPA_AD_IRN, FGPA_AD_IRP, FPGA_SW_VRH
Changed lines of the file:
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@@
 			)
 		)
-		(pin "FGPA_AD_IRP" input
+		(pin "AD_IRP" input
 			(at 207.01 52.07 0)
 			(effects
@@
 			)
 		)
-		(pin "FGPA_AD_ID" input
+		(pin "AD_IRN" input
+			(at 207.01 62.23 0)
+			(effects
+				(font
+					(size 1.27 1.27)
+				)
+				(justify right)
+			)
+		)
+		(pin "AD_IIN" input
+			(at 207.01 59.69 0)
+			(effects
+				(font
+					(size 1.27 1.27)
+				)
+				(justify right)
+			)
+		)
+		(pin "AD_IN" input
+			(at 173.99 52.07 180)
+			(effects
+				(font
+					(size 1.27 1.27)
+				)
+				(justify left)
+			)
+		)
+		(pin "AD_ID" input
 			(at 207.01 54.61 0)
 			(effects
@@
 			)
 		)
-		(pin "AD_COMP" output
-			(at 207.01 57.15 0)
+		(pin "SW_VRH" input
+			(at 207.01 64.77 0)
 			(effects
 				(font
@@
 			)
 		)
-		(pin "FGPA_AD_IIN" input
-			(at 207.01 59.69 0)
+		(pin "AD_CMP" output
+			(at 207.01 57.15 0)
 			(effects
 				(font
-					(size 1.27 1.27)
-				)
-				(justify right)
-			)
-		)
-		(pin "ADIN" input
-			(at 173.99 52.07 180)
-			(effects
-				(font
-					(size 1.27 1.27)
-				)
-				(justify left)
-			)
-		)
-		(pin "FGPA_AD_IRN" input
-			(at 207.01 62.23 0)
-			(effects
-				(font
-					(size 1.27 1.27)
-				)
-				(justify right)
-			)
-		)
-		(pin "FPGA_SW_VRH" input
-			(at 207.01 64.77 0)
-			(effects
-				(font
