File: Hardware/MADC_ARTY/Power.kicad_sch (KiCad schematic)
At the start: 51 parts, among them T1 750319331, U1 TSR_1-2450, U5 UCC25800-Q1, U7 ADP5070AREZ, U8 ADP7142ACPZN, U9 ADP7182ACPZN

Commit message: Schematic
Parts:
- removed C23, C24, C31, C32: 10u/35V, Capacitor_SMD:C_0805_2012Metric, symbol Device:C
- removed D4, D5: DFLS240, Diode_SMD:D_PowerDI-123, symbol Device:D
- removed L2: PA5431.153NLT, DIFF_MEAS:PA5431, symbol Device:L
- removed L3: PM5430.682NLT, DIFF_MEAS:PM5430, symbol Device:L
- removed R17: 0, Resistor_SMD:R_0603_1608Metric, symbol Device:R
- removed R22: 15k, Resistor_SMD:R_0603_1608Metric, symbol Device:R
- removed R24: 113k, Resistor_SMD:R_0603_1608Metric, symbol Device:R
- removed R25: 100k, Resistor_SMD:R_0603_1608Metric, symbol Device:R
- removed R26: 2M15, Resistor_SMD:R_0603_1608Metric, symbol Device:R
- removed R27: 2M1, Resistor_SMD:R_0603_1608Metric, symbol Device:R
- removed R28: 20k, Resistor_SMD:R_0603_1608Metric, symbol Device:R
- removed R29: 10k, Resistor_SMD:R_0603_1608Metric, symbol Device:R
- removed R30: 4k64, Resistor_SMD:R_0603_1608Metric, symbol Device:R
- removed R31: 52k3, Resistor_SMD:R_0603_1608Metric, symbol Device:R
- removed U1: TSR_1-2450, Converter_DCDC:Converter_DCDC_TRACO_TSR-1_THT, symbol Regulator_Switching:TSR_1-2450
- removed U7: ADP5070AREZ, Package_SO:ETSSOP-20-1EP_4.4x6.5mm_P0.65mm_EP3x4.2mm, symbol Regulator_Switching:ADP5070AREZ
- removed U8: ADP7142ACPZN, Package_CSP:LFCSP-6-1EP_2x2mm_P0.65mm_EP1x1.6mm, symbol DIFF_MEAS:ADP7142ACPZN
- removed U9: ADP7182ACPZN, Package_CSP:LFCSP-6-1EP_2x2mm_P0.65mm_EP1x1.6mm, symbol DIFF_MEAS:ADP7182ACPZN
- added U13: NCP1117ST33T3G, Package_TO_SOT_SMD:SOT-223-3_TabPin2, symbol Regulator_Linear:AZ1117-5.0
- added U7: TSR_1-2465, Converter_DCDC:Converter_DCDC_TRACO_TSR-1_THT, symbol Regulator_Switching:TSR_1-2465
- added U8: NCP1117ST50T3G, Package_TO_SOT_SMD:SOT-223-3_TabPin2, symbol Regulator_Linear:AZ1117-5.0
- added U9: SN6505BDBV, Package_TO_SOT_SMD:SOT-23-6, symbol Power_Management:SN6505BDBV
- C13, C14: value 56n/100V -> 56n/50V
- C15: value 47n -> 10u/25V; footprint Capacitor_SMD:C_0603_1608Metric -> Capacitor_SMD:C_1206_3216Metric
- C16, C21: value 1u -> 10u/25V; footprint Capacitor_SMD:C_0603_1608Metric -> Capacitor_SMD:C_1206_3216Metric
- C17: value 68n -> 10u/25V; footprint Capacitor_SMD:C_0603_1608Metric -> Capacitor_SMD:C_1206_3216Metric
- C19, C20: value 4u7/50V -> 10u/50V
- L1: value 74438356033HT -> 74438334056; footprint DIFF_MEAS:L_Wurth_WE-MAPI-4020HT -> (none)
- R21: value 12k -> 0; footprint Resistor_SMD:R_0603_1608Metric -> (none)
Connections:
- net +5V: now also C21.1, R21.2, U8.2 (VO), U9.2 (VCC), U9.5 (EN); no longer C22.1
- net GNDS: now also U5.1 (SYNC)
- net GND: now reaches C17.2
- net GND: now also C14.2, C15.2, C16.2, C18.2, C19.2, C20.2, C21.2, C22.2, D2.2 (A), D3.1 (K), U13.1 (GND), U7.2 (GND), U8.1 (GND), U9.4 (GND), U9.6 (CLK)
- net at C20.1, L1.2: now also U7.1 (Vin)
- net +6V5: now reaches R21.1
- net +6V5: now also C15.1, C17.1, C22.1, U13.3 (VI), U7.3 (Vout), U8.3 (VI); no longer C15.2
- removed net EPAD: C14.2, C15.1, C16.1, C17.1, C18.2, C19.2, C20.2, C21.1, C22.2, D2.2 (A), D3.1 (K)
- new net +3.3V: C16.1, U13.2 (VO)
- no-connect marks 5 -> 1
Other:
- moved on the sheet: C22, L1

Commit message: Schematic
Parts:
- removed C10: 2u2/100V, Capacitor_SMD:C_1206_3216Metric, symbol Device:C
- removed C12: 2u2/50V, Capacitor_SMD:C_0805_2012Metric, symbol Device:C
- removed C14: 56n/50V, Capacitor_SMD:C_0805_2012Metric, symbol Device:C
- removed C15, C16, C17, C21: 10u/25V, Capacitor_SMD:C_1206_3216Metric, symbol Device:C
- removed C18, C8, C9: 10u/50V, Capacitor_SMD:C_1206_3216Metric, symbol Device:C
- removed C7: 1u/50V, Capacitor_SMD:C_0805_2012Metric, symbol Device:C
- removed D1, D2: NRVB0540T1G, Diode_SMD:D_SOD-123, symbol Device:D_Schottky
- removed R15, R16: 4k99, Resistor_SMD:R_0603_1608Metric, symbol Device:R
- removed R18: 30k1, Resistor_SMD:R_0603_1608Metric, symbol Device:R
- removed R19, R20: 100k, Resistor_SMD:R_0805_2012Metric, symbol Device:R
- removed R21: 0, symbol Device:R
- removed T1: 750319331, UCC25800:750319331, symbol UCC25800:750319331
- removed U13: NCP1117ST33T3G, Package_TO_SOT_SMD:SOT-223-3_TabPin2, symbol Regulator_Linear:AZ1117-5.0
- removed U5: UCC25800-Q1, Package_SO:HVSSOP-8-1EP_3x3mm_P0.65mm_EP1.57x1.89mm_ThermalVias, symbol Regulator_Controller:UCC25800
- removed U7: TSR_1-2465, Converter_DCDC:Converter_DCDC_TRACO_TSR-1_THT, symbol Regulator_Switching:TSR_1-2465
- removed U8: NCP1117ST50T3G, Package_TO_SOT_SMD:SOT-223-3_TabPin2, symbol Regulator_Linear:AZ1117-5.0
- removed U9: SN6505BDBV, Package_TO_SOT_SMD:SOT-23-6, symbol Power_Management:SN6505BDBV
- added U27: TSR2-2450, Converter_DCDC:Converter_DCDC_TRACO_TSR2-xxxx_THT, symbol Regulator_Switching:TSR2-2450
- added U5: ADP5070AREZ, Package_SO:ETSSOP-20-1EP_4.4x6.5mm_P0.65mm_EP3x4.2mm, symbol Regulator_Switching:ADP5070AREZ
- added U7: ADP7142ARDZ-3.3, Package_SO:SOIC-8-1EP_3.9x4.9mm_P1.27mm_EP2.29x3mm, symbol Regulator_Linear:ADP7142ARDZ-3.3
- C11: value 2u2/50V -> 10u/25V; footprint Capacitor_SMD:C_0805_2012Metric -> Capacitor_SMD:C_1206_3216Metric
- C13: value 56n/50V -> 10u/25V; footprint Capacitor_SMD:C_0805_2012Metric -> Capacitor_SMD:C_1206_3216Metric
- C7: renamed from C19; value 10u/50V -> 4u7/50V
- C8: renamed from C20; value 10u/50V -> 4u7/50V
- L1: value 74438334056 -> 74479335329247
- renumbered C22 to C9, D3 to D1, R23 to R15
Connections:
- net +6V5 is gone; now on net +5V: C9.1
- net +24V: now also C7.1, L1.1; no longer C11.1
- net +3.3V: now also C13.1, U7.1 (VOUT), U7.2 (VOUT), U7.3 (SENSE/ADJ)
- net +5V: now also C11.1, U27.3 (Vout), U5.11 (EN2), U5.17 (PVIN1), U5.18 (PVINSYS), U5.19 (PVIN2), U5.9 (EN1), U7.5 (EN), U7.7 (VIN), U7.8 (VIN)
- net GND: now also C11.2, C13.2, U27.2 (GND), U5.1 (PGND), U5.15 (AGND), U5.21 (AGND), U7.4 (GND), U7.9 (GND)
- net at C8.1, L1.2: now also U27.1 (Vin)
Other:
- moved on the sheet: C7, C8, C9, L1

Commit message: Schematic
Parts:
- removed U27: TSR2-2450, Converter_DCDC:Converter_DCDC_TRACO_TSR2-xxxx_THT, symbol Regulator_Switching:TSR2-2450
- added C51, C52: 10u/25V, Capacitor_SMD:C_1206_3216Metric, symbol Device:C
- added C53: 0.1u, symbol Device:C
- added C54: 1u/50V, symbol Device:C
- added C55: 47n/50V, symbol Device:C
- added C56: 68n/50V, symbol Device:C
- added C57: 0.1u/50V, symbol Device:C
- added C58, C59, C60, C61, C62, C63, C64: 10u/50V, Capacitor_SMD:C_1206_3216Metric, symbol Device:C
- added D4, D5: V5N3L63HM3/I, symbol Device:D
- added L2: 10u, symbol Device:L
- added L3: 15u, symbol Device:L
- added R42: 10k, symbol Device:R
- added R43, R44, R58: 12k, symbol Device:R
- added R45, R48: 2M4, symbol Device:R
- added R46: 62k, symbol Device:R
- added R47, R52, R55: 39k, symbol Device:R
- added R49: 120k, symbol Device:R
- added R50: 93k, symbol Device:R
- added R51, R54, R57: 620k, symbol Device:R
- added R53: 6k2, symbol Device:R
- added R56: 47k, symbol Device:R
- added R59, R60, R61: 0, symbol Device:R
- added U17: TSR3-2450N, Converter_DCDC:Converter_DCDC_TRACO_TSR2-24xxN_TSR2-24xxxN_THT, symbol Regulator_Switching:TSR3-2450N
- added U26, U27: ADP7182ACPZN, Package_CSP:LFCSP-6-1EP_2x2mm_P0.65mm_EP1x1.6mm, symbol MADC_ARTY:ADP7182ACPZN
- added U4: ADP7142ARDZ, Package_SO:SOIC-8-1EP_3.9x4.9mm_P1.27mm_EP2.29x3mm, symbol Regulator_Linear:ADP7142ARDZ
- renumbered C11 to C10, C13 to C11, U7 to U5, U5 to U6
Connections:
- net +3.3V: now also C52.1
- net +5V: now also C51.1, R42.1, U17.3 (Vout); no longer U6.11 (EN2), U6.9 (EN1)
- net GND: now also U6.4 (SYNC/FREQ), C51.2, C52.2, C53.2, C54.1, C57.2, C58.2, C59.2, C60.2, C61.2, C62.1, C63.1, C64.1, L3.2, R43.1, R44.1, R47.2, R50.2, R53.2, R55.1, R58.1, U17.2 (GND), U26.5 (GND), U27.5 (GND), U4.4 (GND), U4.9 (GND)
- net at U6.12 (COMP2): now also C56.2
- net at U6.13 (FB2): now also R48.2, R49.1
- net at U6.14 (VREF): now also C57.1
- net at U6.16 (VREG): now also C54.2
- net at U6.2 (SW1): now also D4.2 (A), L2.2
- net at U6.20 (SW2): now also D5.1 (K), L3.1
- net at U6.3 (INBK): now also L2.1
- net at U6.7 (FB1): now also R45.2, R46.1
- net at U6.8 (COMP1): now also C55.2
- net at C8.1, L1.2: now also U17.1 (Vin)
- new net: R49.2, R50.1
- new net: R54.1, R55.2, U26.2 (ADJ)
- new net: R54.2, R60.1, U26.1 (VOUT)
- new net: R57.2, R61.1, U27.1 (VOUT)
- new net: R56.2, R57.1, U27.2 (ADJ)
- new net: R51.1, R59.1, U4.1 (VOUT), U4.2 (VOUT)
- new net: C58.1, C61.1, D4.1 (K), R45.1, U4.5 (EN), U4.7 (VIN), U4.8 (VIN)
- new net: R46.2, R47.1
- new net: C56.1, R44.2
- new net: C55.1, R43.2
- new net: R51.2, R52.1, U4.3 (SENSE/ADJ)
- new net: R56.1, R58.2
- new net: R52.2, R53.1
- new net +18V: C60.1, R59.2
- new net -14V: C64.2, R61.2
- new net -18V: C62.2, R60.2
- new net EN1: C53.1, R42.2, U6.11 (EN2), U6.9 (EN1)
- new net EPAD: C59.1, C63.2, D5.2 (A), R48.1, U26.3 (EN), U26.6 (VIN), U26.7 (EPAD), U27.3 (EN), U27.6 (VIN), U27.7 (EPAD)
- no-connect marks 1 -> 5
Other:
- moved on the sheet: C10, C11, C7, C8, C9, L1, U5, U6

Commit message: Schematic
Parts:
- removed U4: ADP7142ARDZ, Package_SO:SOIC-8-1EP_3.9x4.9mm_P1.27mm_EP2.29x3mm, symbol Regulator_Linear:ADP7142ARDZ
- added C65: 10u/50V, Capacitor_SMD:C_1206_3216Metric, symbol Device:C
- added U28: ADP7142ACPZN, Package_CSP:LFCSP-6-1EP_2x2mm_P0.65mm_EP1x1.6mm, symbol MADC_ARTY:ADP7142ACPZN
- C10, C11, C51, C52, C7, C8, C9: footprint Capacitor_SMD:C_1206_3216Metric -> Capacitor_SMD:C_0805_2012Metric
- C53, C54, C55, C56, C57: footprint (none) -> Capacitor_SMD:C_0603_1608Metric
- D4, D5: value V5N3L63HM3/I -> SBR3U40P1Q-7; footprint (none) -> Diode_SMD:D_PowerDI-123
- R42, R43, R44, R45, R46, R47, R48, R49, R50, R51, R52, R53, R54, R55, R56, R57, R58, R59, R60, R61: footprint (none) -> Resistor_SMD:R_0603_1608Metric
Connections:
- net GND is gone; now on net EPAD: C10.2, C11.2, C51.2, C52.2, C53.2, C54.1, C57.2, C58.2, C59.2, C60.2, C61.2, C62.1, C63.1, C64.1, C7.2, C8.2, C9.2, D1.1 (K), L3.2, R43.1, R44.1, R47.2, R50.2, R53.2, R55.1, R58.1, U17.2 (GND), U26.5 (GND), U27.5 (GND), U5.4 (GND), U5.9 (GND), U6.1 (PGND), U6.15 (AGND), U6.21 (AGND), U6.4 (SYNC/FREQ)
- net EPAD: now also C65.1, C65.2, U28.3 (GND), U28.7 (EPAD)
- net at R51.1, R59.1: now also U28.1 (VOUT)
- net at C58.1, C61.1, D4.1 (K)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: now also U28.4 (EN), U28.6 (VIN)
- net at R51.2, R52.1: now also U28.2 (ADJ)
Other:
- moved on the sheet: C57, C60, C61, C62, C63, C64, R51, R52, R53, R54, R55, R56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

Commit message: Schematic
Parts:
- L1: value 74479335329247 -> XFL4020-472MEC; footprint (none) -> Inductor_SMD:L_Coilcraft_XAL4020-XXX
- L2: value 10u -> XAL4040-103MEC; footprint (none) -> Inductor_SMD:L_Coilcraft_XAL4040-XXX
- L3: value 15u -> XAL5050-153MEC; footprint (none) -> Inductor_SMD:L_Coilcraft_XAL5050-XXX
Other:
- moved on the sheet: C10, C11, C51, C52, C53, C54, C55, C56, C57, C58, C59, C60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

Commit message: PCB and Schematic
Parts:
- added J5: Conn_01x02, symbol Connector_Generic:Conn_01x02
- added TP13, TP14, TP15, TP16, TP17, TP18: TestPoint, symbol Connector:TestPoint
- renumbered C56 to C10, C9 to C11, C51 to C12, C57 to C13, C10 to C14, C11 to C15, C58 to C16, C59 to C17, C52 to C18, C61 to C19, C63 to C20, C65 to C21, C60 to C22, C62 to C23, C64 to C24, C7 to C5, C53 to C6, C8 to C7, C55 to C8, C54 to C9, D5 to D2, D4 to D3, L3 to L2, L2 to L3, R42 to R11, R43 to R12, R44 to R13, R15 to R14, R48 to R15, R45 to R16, R46 to R17, R49 to R18, R47 to R19, R50 to R20, R51 to R21, R52 to R22, R53 to R23, R55 to R24, R54 to R25, R58 to R26, R56 to R27, R57 to R28, R59 to R29, R60 to R30, R61 to R31, U17 to U3, U6 to U4, U28 to U6, U26 to U7, U27 to U8
Connections:
- net +24V: now also J5.1 (Pin_1)
- net EPAD: now also J5.2 (Pin_2), TP13.1, TP18.1
- net at R25.2, R30.1, U7.1 (VOUT): now also TP15.1
- net at R28.2, R31.1, U8.1 (VOUT): now also TP14.1
- net at R21.1, R29.1, U6.1 (VOUT): now also TP16.1
- net at C16.1, C19.1, D3.1 (K)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: now also TP17.1
Other:
- moved on the sheet: C11, C12, C14, C5, C7, D1, L1, R14, U3

Commit message: PCB
Parts:
- removed TP18: TestPoint, symbol Connector:TestPoint
- removed U6: ADP7142ACPZN, Package_CSP:LFCSP-6-1EP_2x2mm_P0.65mm_EP1x1.6mm, symbol MADC_ARTY:ADP7142ACPZN
- added D1: DZ2S100X0L, Diode_SMD:D_SOD-523, symbol Diode:DZ2S100X0L
- added Q7: SiS443DN, Package_SO:Vishay_PowerPAK_1212-8_Single, symbol Transistor_FET:SiS443DN
- added R12: 0, Resistor_SMD:R_0603_1608Metric, symbol Device:R
- added R13: 100k, Resistor_SMD:R_0603_1608Metric, symbol Device:R
- added TP7: TestPoint, TestPoint:TestPoint_Keystone_5010-5014_Multipurpose, symbol Connector:TestPoint
- added TP9: TestPoint, TestPoint:TestPoint_Pad_D2.0mm, symbol Connector:TestPoint
- added U6: ADP7142ARDZ, Package_SO:SOIC-8-1EP_3.9x4.9mm_P1.27mm_EP2.29x3mm, symbol Regulator_Linear:ADP7142ARDZ
- J3: renamed from J5; footprint (none) -> TerminalBlock_Phoenix:TerminalBlock_Phoenix_MPT-0,5-2-2.54_1x02_P2.54mm_Horizontal
- TP10: renamed from TP16; footprint (none) -> TestPoint:TestPoint_Pad_D2.0mm
- TP11: renamed from TP15; footprint (none) -> TestPoint:TestPoint_Pad_D2.0mm
- TP12: renamed from TP14; footprint (none) -> TestPoint:TestPoint_Pad_D2.0mm
- TP6: renamed from TP13; footprint (none) -> TestPoint:TestPoint_Keystone_5010-5014_Multipurpose
- TP8: renamed from TP17; footprint (none) -> TestPoint:TestPoint_Pad_D2.0mm
- renumbered D1 to D2, D2 to D3, D3 to D4, R12 to R14, R13 to R15, R14 to R16, R15 to R17, R16 to R18, R17 to R19, R18 to R20, R19 to R21, R20 to R22, R21 to R23, R22 to R24, R23 to R25, R24 to R26, R25 to R27, R26 to R28, R27 to R29, R28 to R30, R29 to R31, R30 to R32, R31 to R33
Connections:
- net +18V: now also TP10.1
- net +24V: now also D1.1 (K), Q7.1 (S), Q7.2 (S), Q7.3 (S), R12.2; no longer J3.1 (Pin_1)
- net -14V: now also TP12.1
- net -18V: now also TP11.1
- net at R27.2, R32.1, U7.1 (VOUT): no longer TP11.1
- net at R30.2, R33.1, U8.1 (VOUT): no longer TP12.1
- net at R23.1, R31.1: now also U6.1 (VOUT), U6.2 (VOUT); no longer TP10.1
- net at C16.1, C19.1, D4.1 (K)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: now also U6.5 (EN), U6.7 (VIN), U6.8 (VIN)
- net at R23.2, R24.1: now also U6.3 (SENSE/ADJ)
- net EPAD renamed GND
- net GND: now also R13.2, TP7.1, U6.4 (GND), U6.9 (GND); no longer C17.1, C20.2, C21.2, D3.2 (A), R17.1, U7.3 (EN), U7.6 (VIN), U7.7 (EPAD), U8.3 (EN), U8.6 (VIN), U8.7 (EPAD)
- new net: D1.2 (A), Q7.4 (G), R13.1
- new net: J3.1 (Pin_1), Q7.5 (D), R12.1
- new net: C17.1, C20.2, C21.2, D3.2 (A), R17.1, TP9.1, U7.3 (EN), U7.6 (VIN), U7.7 (EPAD), U8.3 (EN), U8.6 (VIN), U8.7 (EPAD)
Other:
- moved on the sheet: C10, C11, C12, C13, C14, C15, C16, C17, C18, C19, C20, C21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

Commit message: PCB and schematic
Parts:
- TP10, TP11, TP12, TP8, TP9: now left out of the parts list
Connections:
- net EN1: no longer names the net of C6.1, R11.2, U4.11 (EN2), U4.9 (EN1)
