File: Hardware/MADC_ARTY/Power.kicad_sch (KiCad schematic)
At the start: 65 parts, among them J3 Conn_01x02, Q7 SiS443DN, U3 TSR3-2450N, U4 ADP5070AREZ, U5 ADP7142ARDZ-3.3, U6 ADP7142ARDZ, U7 ADP7182ACPZN, U8 ADP7182ACPZN

Commit message: BOM
Parts:
- removed D1: DZ2S100X0L, Diode_SMD:D_SOD-523, symbol Diode:DZ2S100X0L
- added D1: BZX84C10LT1G, Package_TO_SOT_SMD:SOT-23, symbol Diode:BZX84Cxx
- added D2: 1N4148W, Diode_SMD:D_SOD-123, symbol Diode:1N4148W
- added Q8: MMBT3904VL, Package_TO_SOT_SMD:SOT-23, symbol Transistor_BJT:MMBT3904
- added R16: 100k, Resistor_SMD:R_0603_1608Metric, symbol Device:R
- added R80: 6k2, Resistor_SMD:R_0603_1608Metric, symbol Device:R
- J3: value Conn_01x02 -> 1715721; footprint TerminalBlock_Phoenix:TerminalBlock_Phoenix_MPT-0,5-2-2.54_1x02_P2.54mm_Horizontal -> TerminalBlock_Phoenix:TerminalBlock_Phoenix_MKDS-1,5-2_1x02_P5.00mm_Horizontal
- TP6, TP7: now left out of the parts list
- renumbered D2 to D3, D3 to D4, D4 to D5, R16 to R17, R17 to R18, R18 to R19, R19 to R20, R20 to R21, R21 to R22, R22 to R23, R23 to R24, R24 to R25, R25 to R26, R26 to R27, R27 to R28, R28 to R29, R29 to R30, R30 to R31, R31 to R32, R32 to R33, R33 to R34
Connections:
- net +24V: now also D1.3 (K), D2.2 (A), Q8.2 (E)
- net GND: now also R16.2, R80.2; no longer R27.1
- net at Q7.4 (G), R13.1: now also D1.1 (A), Q8.3 (C)
- new net: R27.1, R80.1
- new net: D2.1 (K), Q8.1 (B), R16.1
Other:
- moved on the sheet: J3, Q7, R12, R13, R26
