File: Hardware/MADC_ARTY/ADC.kicad_sch (KiCad schematic)
At the start: 49 parts, among them U15 DG211BDQ, U16 OPA2192, U17 DG419xY, U18 LT5400-2, U19 ADR1399KEZ, U20 LT5400-6, U21 OPA177GS, U22 OPA140, U23 LT5400-1, U24 OPA2192, U25 OPA192, U26 LM311

Commit message: Schematic
Parts:
- removed C14, C33: 0.1u, Capacitor_SMD:C_0603_1608Metric, symbol Device:C
- removed R24: 62, Resistor_SMD:R_0603_1608Metric, symbol Device:R
- removed R38: 12k, Resistor_SMD:R_0603_1608Metric, symbol Device:R
- removed U16, U24: OPA2192, Package_SO:SOIC-8_3.9x4.9mm_P1.27mm, symbol ADC_TEST:OPA2192
- removed unit 1 of U17
- removed U19: ADR1399KEZ, Package_LCC:Analog_LCC-8_5x5mm_P1.27mm, symbol Reference_Voltage:ADR1399KEZ
- removed U20: LT5400-6, Package_SO:MSOP-8-1EP_3x3mm_P0.65mm_EP1.73x1.85mm_ThermalVias, symbol ADC_TEST:LT5400-5k-1k
- removed U21: OPA177GS, Package_SO:SOIC-8_3.9x4.9mm_P1.27mm, symbol ADC_TEST:OPA177
- removed U23: LT5400-1, Package_SO:MSOP-8-1EP_3x3mm_P0.65mm_EP1.73x1.85mm_ThermalVias, symbol ADC_TEST:LT5400-10k-10k
- added C26, C27, C28, C29: 0.1u, Capacitor_SMD:C_0603_1608Metric, symbol Device:C
- added U14: LT5400-6, Package_SO:MSOP-8-1EP_3x3mm_P0.65mm_EP1.73x1.85mm_ThermalVias, symbol ADC_TEST:LT5400-5k-1k
- added unit 1 of U16
- added U19: LT5400-1, Package_SO:MSOP-8-1EP_3x3mm_P0.65mm_EP1.73x1.85mm_ThermalVias, symbol ADC_TEST:LT5400-10k-10k
- added U25: OPA2192, Package_SO:VSSOP-8_3x3mm_P0.65mm, symbol Amplifier_Operational:OPA2197xDGK
- renumbered C31 to C24, C32 to C25, C27 to C30, C28 to C31, C30 to C32, C15 to C33, C16 to C34, C17 to C35, C18 to C36, C19 to C37, C20 to C38, C21 to C39, C22 to C40, C23 to C41, C24 to C42, C25 to C43, C26 to C44, C29 to C45, R25 to R24, R26 to R25, R27 to R26, R28 to R27, R29 to R28, R30 to R29, R31 to R30, R33 to R31, R34 to R33, R35 to R34, R36 to R35, R37 to R36, U18 to U15, U17 to U16, U15 to U18, U22 to U20, U25 to U21, U26 to U22
Connections:
- net +18V: now also C26.1, U25.8 (V+)
- net -14V: no longer U16.7 (V-), U18.4 (V-)
- net -18V: now also U16.7 (V-), U18.4 (V-), C27.1, C28.1, C29.1, U25.4 (V-)
- net FPGA_SW_VRH: now also U16.6
- net GND: now also C26.2, C27.2, C28.2, C29.2, U14.6, U14.9 (EP), U19.9 (EP), U25.5 (+)
- net VREF+: now also U19.1, U19.2, U25.7
- net VREF-: now also U19.3, U19.4, U25.1, U25.2 (-)
- new net: U16.1, U25.3 (+)
- new net: U14.7, U14.8, U16.2
- new net: U14.5, U16.8
- new net: U19.5, U19.6, U19.7, U19.8, U25.6 (-)
- new net: U14.1, U14.4
- new net: U14.2, U14.3
- no-connect marks 3 -> 1
Other:
- moved on the sheet: C24, C25, C30, C31, C32, U16B, U18E

Commit message: Schematic
Parts:
- C35, C36, C39, C40: footprint (none) -> Capacitor_SMD:C_0805_2012Metric
- C37, C38, C42, C43: footprint (none) -> Capacitor_SMD:C_0603_1608Metric
Changed lines of the file:
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@@
 			)
 		)
-		(property "Footprint" ""
+		(property "Footprint" "Capacitor_SMD:C_0603_1608Metric"
 			(at 171.45 67.6148 0)
 			(effects
@@
 			)
 		)
-		(property "Footprint" ""
+		(property "Footprint" "Capacitor_SMD:C_0603_1608Metric"
 			(at 220.98 65.0748 0)
 			(effects
@@
 			)
 		)
-		(property "Footprint" ""
+		(property "Footprint" "Capacitor_SMD:C_0603_1608Metric"
 			(at 171.45 35.8648 0)
 			(effects
@@
 			)
 		)
-		(property "Footprint" ""
+		(property "Footprint" "Capacitor_SMD:C_0805_2012Metric"
 			(at 161.29 35.8648 0)
 			(effects
@@
 			)
 		)
-		(property "Footprint" ""
+		(property "Footprint" "Capacitor_SMD:C_0603_1608Metric"
 			(at 220.98 33.3248 0)
 			(effects
@@
 			)
 		)
-		(property "Footprint" ""
+		(property "Footprint" "Capacitor_SMD:C_0805_2012Metric"
 			(at 161.29 67.6148 0)
 			(effects
@@
 			)
 		)
-		(property "Footprint" ""
+		(property "Footprint" "Capacitor_SMD:C_0805_2012Metric"
 			(at 210.82 33.3248 0)
 			(effects
@@
 			)
 		)
-		(property "Footprint" ""
+		(property "Footprint" "Capacitor_SMD:C_0805_2012Metric"
 			(at 210.82 65.0748 0)
 			(effects

Commit message: PCB and Schematic
Parts:
- added TP3, TP4, TP5, TP6, TP7, TP8, TP9: TestPoint, symbol Connector:TestPoint
- renumbered C24 to C33, C25 to C34, C26 to C35, C27 to C36, C28 to C37, C29 to C38, C30 to C39, C31 to C40, C32 to C41, C33 to C42, C34 to C43, C35 to C44, C36 to C45, C37 to C46, C38 to C47, C39 to C48, C40 to C49, C41 to C50, C42 to C51, C43 to C52, C44 to C53, C45 to C54, D2 to D4, D3 to D5, R24 to R42, R25 to R43, R26 to R44, R27 to R45, R28 to R46, R29 to R47, R30 to R48, R31 to R49, R32 to R50, R33 to R51, R34 to R52, R35 to R53, R36 to R54, U25 to U17
Connections:
- net AD_COMP: now also TP3.1
- net VREF+: now also TP9.1
- net VREF-: now also TP8.1
- net at C42.2, C43.2, U18.10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: now also TP5.1
- net at C42.1, C43.1, R44.2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: now also TP4.1
- net at C50.1, D4.1 (K), D5.2 (A)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: now also TP7.1
- net at C50.2, D4.2 (A), D5.1 (K)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: now also TP6.1
Other:
- moved on the sheet: C42, C43, C44, C45, C46, C47, C48, C49, C50, C51, C52, C53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

Commit message: PCB
Parts:
- removed TP3: TestPoint, symbol Connector:TestPoint
- TP15: renamed from TP5; footprint (none) -> TestPoint:TestPoint_Pad_D2.0mm
- TP16: renamed from TP8; footprint (none) -> TestPoint:TestPoint_Pad_D2.0mm
- TP17: renamed from TP4; footprint (none) -> TestPoint:TestPoint_Pad_D2.0mm
- TP18: renamed from TP6; footprint (none) -> TestPoint:TestPoint_Pad_D2.0mm
- TP19: renamed from TP9; footprint (none) -> TestPoint:TestPoint_Pad_D2.0mm
- TP20: renamed from TP7; footprint (none) -> TestPoint:TestPoint_Pad_D2.0mm
- renumbered D4 to D5, D5 to D6, R42 to R44, R43 to R45, R44 to R46, R45 to R47, R46 to R48, R47 to R49, R48 to R50, R49 to R51, R50 to R52, R51 to R53, R52 to R54, R53 to R55, R54 to R56, U18 to U17, U17 to U18
Connections:
- net -7V: now reaches U14.5, U16.8

Commit message: MADC module send to production
Parts:
- removed C33, C34, C35, C36, C37, C38, C39, C40, C41, C54: 0.1u, Capacitor_SMD:C_0603_1608Metric, symbol Device:C
- removed C42: 23PS222, Capacitor_THT:C_Axial_L12.0mm_D6.5mm_P15.00mm_Horizontal, symbol Device:C
- removed C43: 2n2/SMD, Capacitor_SMD:C_0603_1608Metric, symbol Device:C
- removed C44, C45, C48, C49: 10u/35V, Capacitor_SMD:C_0805_2012Metric, symbol Device:C
- removed C46, C47, C51, C52: 1u/35V, Capacitor_SMD:C_0603_1608Metric, symbol Device:C
- removed C50: 33p, Capacitor_SMD:C_0603_1608Metric, symbol Device:C
- removed C53: DNP, Capacitor_SMD:C_0603_1608Metric, symbol Device:C
- removed D5, D6: BAV21W, Diode_SMD:D_SOD-123, symbol Device:D
- removed R44, R45, R48, R49, R53: 10, Resistor_SMD:R_0603_1608Metric, symbol Device:R
- removed R46: 12k/.05%, Resistor_SMD:R_0603_1608Metric, symbol Device:R
- removed R47: 62k, Resistor_SMD:R_0603_1608Metric, symbol Device:R
- removed R50: 0, Resistor_SMD:R_0603_1608Metric, symbol Device:R
- removed R51: 3k9/.05%, Resistor_SMD:R_0603_1608Metric, symbol Device:R
- removed R52: 620/.05%, Resistor_SMD:R_0603_1608Metric, symbol Device:R
- removed R54: 62, Resistor_SMD:R_0603_1608Metric, symbol Device:R
- removed R55: 39k, Resistor_SMD:R_0603_1608Metric, symbol Device:R
- removed R56: 3k9, Resistor_SMD:R_0603_1608Metric, symbol Device:R
- removed TP15, TP16, TP17, TP18, TP19, TP20: TestPoint, TestPoint:TestPoint_Pad_D2.0mm, symbol Connector:TestPoint
- removed U14: LT5400-6, Package_SO:MSOP-8-1EP_3x3mm_P0.65mm_EP1.73x1.85mm_ThermalVias, symbol ADC_TEST:LT5400-5k-1k
- removed U15: LT5400-2, Package_SO:MSOP-8-1EP_3x3mm_P0.65mm_EP1.73x1.85mm_ThermalVias, symbol ADC_TEST:LT5400-100k-100k
- removed U16: DG419xY, Package_SO:SOIC-8_3.9x4.9mm_P1.27mm, symbol Analog_Switch:DG419xY
- removed U17: DG211BDQ, Package_SO:SOIC-16_3.9x9.9mm_P1.27mm, symbol ADC_TEST:DG211
- removed U18: OPA2192, Package_SO:VSSOP-8_3x3mm_P0.65mm, symbol Amplifier_Operational:OPA2197xDGK
- removed U19: LT5400-1, Package_SO:MSOP-8-1EP_3x3mm_P0.65mm_EP1.73x1.85mm_ThermalVias, symbol ADC_TEST:LT5400-10k-10k
- removed U20: OPA140, Package_SO:SOIC-8_3.9x4.9mm_P1.27mm, symbol ADC_TEST:OPA140
- removed U21: OPA192, Package_SO:SOIC-8_3.9x4.9mm_P1.27mm, symbol ADC_TEST:OPA192
- removed U22: LM311, Package_SO:SOIC-8_3.9x4.9mm_P1.27mm, symbol Comparator:LM311
Connections:
- no-connect marks 1 -> 0

Commit message: PCB and schematic
Parts:
- added C48, C49: 0.1u, Capacitor_SMD:C_0603_1608Metric, symbol Device:C
- added R66, R67, R68, R69, R71, R73: 0, Resistor_SMD:R_0603_1608Metric, symbol Device:R
- added R72: 1k, Resistor_SMD:R_0603_1608Metric, symbol Device:R
- added U21: MADC, MADC:MADC, symbol MADC_ARTY:MADC
- added U22: SN74LVC1T45DBV, Package_TO_SOT_SMD:SOT-23-6, symbol Logic_LevelTranslator:SN74LVC1T45DBV
Connections:
- new net: R73.2, U21.3 (AD_CMP), U22.4 (B)
- new net: R66.2, R67.2, U21.16 (VREF)
- new net: R71.2, R72.2, U22.5 (DIR)
- new net: R68.2, R69.2, U21.15 (VEE)
- new net +18V: U21.14 (VCC)
- new net +3.3V: C49.1, U21.2 (+3V3), U22.6 (VCCB)
- new net +3.3VP: C48.1, R72.1, U22.1 (VCCA)
- new net +7V: R66.1
- new net -14V: R69.1
- new net -18V: R68.1
- new net -7V: R67.1
- new net AD_CMP: R73.1, U22.3 (A)
- new net AD_ID: U21.8 (AD_ID)
- new net AD_IIN: U21.6 (AD_IIN)
- new net AD_IN: U21.11 (AD_IN), U21.13 (AD_IN)
- new net AD_IRN: U21.4 (AD_IRN)
- new net AD_IRP: U21.7 (AD_IRP)
- new net GND: C48.2, C49.2, R71.1, U21.1 (GNDD), U21.10 (GNDA), U21.12 (GNDA), U21.9 (GNDA), U22.2 (GND)
- new net SW_VRH: U21.5 (SW_VRH)

Commit message: BOM
Parts:
- renumbered C48 to C35, C49 to C36, R66 to R50, R67 to R51, R68 to R52, R69 to R53, R73 to R54, R71 to R55, R72 to R56, U21 to U15, U22 to U16
