File: Hardware/MADC_ARTY/MADC_ARTY.kicad_pcb (KiCad board)
At the start: 2 copper layers, 177 parts, among them J1 Conn_01x01, J2 Conn_01x01, J3 71764-0012, J4 71764-0012, Q1 MMBT6429, Q10 MMBF4392, Q11 MMBT6429, Q12 MMBT6429, Q2 JFE2140D, Q3 MMBT6429, Q4 MMBF4392, Q5 MMBT6429, Q6 MMBT6429, Q7 MMBT6429, Q8 JFE2140D, Q9 MMBT6429, U1 OPA2192, U10 ADG419BRM, U11 ADG419BRM, U12 ADG419BRM, U13 ADG419BRM, U14 LT5400-6, U15 LT5400-2, U16 DG419xY, U17 TSR3-2450N, U18 DG211BDQ, U19 LT5400-1, U2 OPA4192IPW, U20 OPA140, U21 OPA192, U22 LM311, U23 OPA2192, U24 ADR1399KEZ, U25 OPA2192, U26 ADP7182ACPZN, U27 ADP7182ACPZN, U28 ADP7142ACPZN, U3 OPA4192IPW, U5 ADP7142ARDZ-3.3, U6 ADP5070AREZ, U7 AQY212G3HS, U8 AQY212G3HS, U9 AD8422ARMZ

Commit message: Schematic
Parts:
- added L1: XFL4020-472MEC, Inductor_SMD:L_Coilcraft_XAL4020-XXX, F.Cu at (241.3, 75.5)
- added L2: XAL4040-103MEC, Inductor_SMD:L_Coilcraft_XAL4040-XXX, F.Cu at (243.8, 87.0)
- added L3: XAL5050-153MEC, Inductor_SMD:L_Coilcraft_XAL5050-XXX, F.Cu at (234.9, 76.2)
- added R63: 0, Resistor_SMD:R_0603_1608Metric, F.Cu at (236.9, 85.3)
- added R64: 0, Resistor_SMD:R_0603_1608Metric, F.Cu at (115.3, 63.4)
- added R65: 10k, Resistor_SMD:R_0603_1608Metric, F.Cu at (236.9, 90.3)
- moved C33 116.3 mm to (207.2, 70.5)
- moved C16 93.2 mm to (110.6, 64.3), turned to 90 degrees
- moved R20 89.4 mm to (115.4, 67.6), turned to 90 degrees
- moved C20 88.5 mm to (112.9, 71.6)
- moved C12 85.1 mm to (110.6, 71.0), turned to -90 degrees
- moved U10 80.0 mm to (112.9, 67.6), turned to -90 degrees
- moved U12 79.5 mm to (119.6, 67.6), turned to -90 degrees
- moved U17 73.1 mm to (136.3, 104.0)
- moved Q2 36.3 mm to (198.4, 103.9)
- moved C18 25.4 mm to (203.9, 128.5)
- moved C21 25.4 mm to (203.9, 136.0)
- moved C36 25.4 mm to (137.3, 88.0)
- moved C50 25.4 mm to (143.0, 120.6)
- moved R18 25.4 mm to (143.0, 128.1)
- moved C10 25.4 mm to (172.3, 70.9)
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Connections:
- J3 pad 5: /Block Diagram/Auto Zero/AZ1_CTR -> /Block Diagram/PMOD/AZ_CTR
- J3 pad 6: /Block Diagram/Auto Zero/AZ2_CTR -> unconnected-(J3-Pin_6-Pad6)
- J3 pad 7: /Block Diagram/Gain/GAIN_x10 -> unconnected-(J3-Pin_7-Pad7)
- J3 pad 8: /Block Diagram/Gain/GAIN_x100 -> unconnected-(J3-Pin_8-Pad8)
- J4 pad 10: unconnected-(J4-Pin_10-Pad10) -> /Block Diagram/ADC/AD_COMP
- J4 pad 11: unconnected-(J4-Pin_11-Pad11) -> /Block Diagram/Gain/GAIN_x10
- J4 pad 12: /Block Diagram/ADC/AD_COMP -> /Block Diagram/Gain/GAIN_x100
- Q8 pad 3: (no net) -> unconnected-(Q8C-VCH-Pad3)
- Q8 pad 7: (no net) -> unconnected-(Q8C-VCL-Pad7)
- U10 pad 6: /Block Diagram/Auto Zero/AZ1_CTR -> /Block Diagram/Auto Zero/AZ_CTR
- U11 pad 6: /Block Diagram/Auto Zero/AZ1_CTR -> /Block Diagram/Auto Zero/AZ_CTR
- U12 pad 6: /Block Diagram/Auto Zero/AZ2_CTR -> /Block Diagram/Auto Zero/AZ_CTR
- U13 pad 6: /Block Diagram/Auto Zero/AZ2_CTR -> /Block Diagram/Auto Zero/AZ_CTR

Commit message: PCB and Schematic
Parts:
- removed the C1 at (171.2, 112.7)
- removed the C12 at (110.6, 71.0)
- removed the C13 at (199.9, 131.0)
- removed the C16 at (110.6, 64.3)
- removed the C17 at (199.9, 141.1)
- removed the C20 at (112.9, 71.6)
- removed the C21 at (203.9, 136.0)
- removed the C4 at (171.2, 120.2)
- removed the R10 at (183.2, 112.7)
- removed the R11 at (183.2, 115.2)
- removed the R12 at (183.2, 117.7)
- removed the R13 at (183.2, 120.2)
- removed the R14 at (183.2, 122.7)
- removed the R20 at (115.4, 67.6)
- removed the R22 at (207.9, 133.5)
- removed the R9 at (179.2, 122.7)
- removed the U10 at (112.9, 67.6)
- removed the U12 at (119.6, 67.6)
- removed the U3 at (164.8, 121.3)
- added C58: 0.1u, Capacitor_SMD:C_0603_1608Metric, F.Cu at (110.2, 86.6)
- added C59: 0.1u, Capacitor_SMD:C_0603_1608Metric, F.Cu at (119.6, 86.6)
- added C60: 0.1u, Capacitor_SMD:C_0603_1608Metric, F.Cu at (118.1, 86.6)
- added C61: 0.1u, Capacitor_SMD:C_0603_1608Metric, F.Cu at (127.5, 86.6)
- added C62: 0.1u, Capacitor_SMD:C_0603_1608Metric, F.Cu at (115.6, 89.2)
- added C63: 0.1u, Capacitor_SMD:C_0603_1608Metric, F.Cu at (125.0, 89.2)
- added C64: 0.1u, Capacitor_SMD:C_0603_1608Metric, F.Cu at (146.6, 95.5)
- added C65: 0.1u, Capacitor_SMD:C_0603_1608Metric, F.Cu at (143.1, 87.4)
- added C66: 0.1u, Capacitor_SMD:C_0603_1608Metric, F.Cu at (152.5, 87.4)
- added C67: 0.1u, Capacitor_SMD:C_0603_1608Metric, F.Cu at (149.2, 90.4)
- added R3: 0, Resistor_SMD:R_0603_1608Metric, B.Cu at (147.8, 72.9)
- added R41: 0, Resistor_SMD:R_0603_1608Metric, F.Cu at (121.9, 65.0)
- added R5: 0, Resistor_SMD:R_0603_1608Metric, F.Cu at (143.9, 73.9)
- added R60: 10k, Resistor_SMD:R_0603_1608Metric, F.Cu at (115.8, 84.1)
- added R61: 0, Resistor_SMD:R_0603_1608Metric, F.Cu at (112.5, 84.1)
- added R62: 10k, Resistor_SMD:R_0603_1608Metric, F.Cu at (119.6, 89.2)
- added R63: 10k, Resistor_SMD:R_0603_1608Metric, F.Cu at (125.2, 84.1)
- added R65: 14k7, Resistor_SMD:R_0603_1608Metric, F.Cu at (153.0, 91.3)
- added R66: 21k5/0.125W, Resistor_SMD:R_0603_1608Metric, F.Cu at (130.4, 78.9)
- added R67: 0, Resistor_SMD:R_0603_1608Metric, B.Cu at (147.8, 91.9)
- added R68: 21k5/0.125W, Resistor_SMD:R_0603_1608Metric, F.Cu at (153.0, 92.8)
- added R69: 0, Resistor_SMD:R_0603_1608Metric, F.Cu at (143.9, 93.0)
- added R70: 2k/0.1%, Resistor_SMD:R_0603_1608Metric, F.Cu at (140.0, 84.1)
- added R71: 2k/0.1%, Resistor_SMD:R_0603_1608Metric, F.Cu at (153.0, 94.4)
- added R72: 0, Resistor_SMD:R_0603_1608Metric, B.Cu at (147.8, 93.6)
- added R73: 2k/0.1%, Resistor_SMD:R_0603_1608Metric, F.Cu at (140.0, 89.7)
- added R74: 21k5/0.125W, Resistor_SMD:R_0603_1608Metric, F.Cu at (131.6, 91.1)
- added U25: ADG419BRM, Package_SO:MSOP-8_3x3mm_P0.65mm, F.Cu at (114.2, 86.6)
- added U26: ADG419BRM, Package_SO:MSOP-8_3x3mm_P0.65mm, F.Cu at (123.6, 86.6)
- added U27: OPA2192, Package_SO:VSSOP-8_3x3mm_P0.65mm, F.Cu at (147.8, 93.0)
- added U28: OPA4192IPW, Package_SO:TSSOP-14_4.4x5mm_P0.65mm, F.Cu at (147.8, 86.6)
- Q12, Q6: moved to B.Cu
- Q2: renamed from Q1; moved to B.Cu
- Q7: value MMBT6429 -> JFE2140D; footprint Package_TO_SOT_SMD:SOT-23 -> Package_SO:SOIC-8_3.9x4.9mm_P1.27mm
- Q8: value JFE2140D -> MMBT6429; footprint Package_SO:SOIC-8_3.9x4.9mm_P1.27mm -> Package_TO_SOT_SMD:SOT-23; moved to B.Cu
- R32: renamed from R16; moved to B.Cu
- R33: renamed from R17; moved to B.Cu
- R8: value 14k7 -> 0; moved to B.Cu
- moved R38 126.0 mm to (112.5, 65.0), turned to 180 degrees
- moved R39 119.0 mm to (119.6, 70.1), turned to 180 degrees
- moved R37 113.3 mm to (115.8, 65.0), turned to 180 degrees
- moved C27 111.8 mm to (110.2, 67.6), turned to 90 degrees
- moved C29 111.4 mm to (118.1, 67.6), turned to -90 degrees
- moved R40 109.0 mm to (125.2, 65.0), turned to 180 degrees
- moved C30 106.0 mm to (127.5, 67.6), turned to -90 degrees
- moved C31 105.5 mm to (115.6, 70.1), turned to 180 degrees
- moved C28 105.5 mm to (119.6, 67.6), turned to 90 degrees
- moved U12 104.1 mm to (114.2, 67.6)
- moved U13 103.6 mm to (123.6, 67.6)
- moved C32 99.8 mm to (125.0, 70.1), turned to 180 degrees
- moved C42 90.7 mm to (291.1, 35.9)
- moved R20 82.7 mm to (258.8, 25.5)
- moved R21 82.7 mm to (258.8, 28.0)
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- renumbered C2 to C1, C56 to C10, C9 to C11, C51 to C12, C57 to C13, C10 to C14, C11 to C15, C58 to C16, C59 to C17, C52 to C18, C61 to C19, C3 to C2, C63 to C20, C65 to C21, C60 to C22, C62 to C23, C64 to C24, C49 to C25, C50 to C26, C18 to C27, C19 to C28, C22 to C29, C5 to C3, C23 to C30, C14 to C31, C15 to C32, C24 to C33, C25 to C34, C26 to C35, C27 to C36, C28 to C37, C29 to C38, C30 to C39, C6 to C4, C31 to C40, C32 to C41, C33 to C42, C34 to C43, C35 to C44, C36 to C45, C37 to C46, C38 to C47, C39 to C48, C40 to C49, C7 to C5, C41 to C50, C42 to C51, C43 to C52, C44 to C53, C45 to C54, C46 to C55, C47 to C56, C48 to C57, C53 to C6, C8 to C7, C55 to C8, C54 to C9, D5 to D2, D4 to D3, D2 to D4, D3 to D5, L3 to L2, L2 to L3, Q2 to Q1, R7 to R10, R42 to R11, R43 to R12, R44 to R13, R15 to R14, R48 to R15, R45 to R16, R46 to R17, R49 to R18, R47 to R19, R50 to R20, R51 to R21, R52 to R22, R53 to R23, R55 to R24, R54 to R25, R58 to R26, R56 to R27, R57 to R28, R59 to R29, R60 to R30, R61 to R31, R18 to R34, R19 to R35, R62 to R36, R21 to R37, R63 to R38, R65 to R39, R3 to R4, R23 to R40, R24 to R42, R25 to R43, R26 to R44, R27 to R45, R28 to R46, R29 to R47, R30 to R48, R31 to R49, R32 to R50, R33 to R51, R34 to R52, R35 to R53, R36 to R54, R37 to R55, R38 to R56, R39 to R57, R40 to R58, R41 to R59, R4 to R6, R5 to R7, R6 to R9, U8 to U10, U9 to U11, U11 to U12, U25 to U17, U17 to U3, U6 to U4, U28 to U6, U26 to U7, U27 to U8, U7 to U9
Connections:
- net /Block Diagram/Analog Channels/OUT_P renamed /Block Diagram/Analog Channels/OUT
- J1 pad 1: /Block Diagram/Auto Zero/AIN_P -> /Block Diagram/Auto Zero/AIN
- J2 pad 1: /Block Diagram/Auto Zero/AIN_N -> /Block Diagram/Auto Zero1/AIN
- J3 pad 5: /Block Diagram/PMOD/AZ_CTR -> /Block Diagram/Auto Zero/AZ_CTR
- Q1 pad 4: /Block Diagram/Analog Channels/IN_P -> /Block Diagram/Analog Channels/IN
- Q7 pad 1: Net-(Q7-B) -> Net-(Q8-C)
- Q7 pad 2: Net-(Q7-E) -> Net-(Q10-S)
- Q7 pad 3: Net-(Q7-C) -> unconnected-(Q7C-VCH-Pad3)
- Q8 pad 1: Net-(Q7-C) -> Net-(Q8-B)
- Q8 pad 2: Net-(Q10-S) -> Net-(Q8-E)
- Q8 pad 3: unconnected-(Q8C-VCH-Pad3) -> Net-(Q8-C)
- Q9 pad 1: Net-(Q7-E) -> Net-(Q8-E)
- Q9 pad 3: Net-(Q7-C) -> Net-(Q8-C)
- R38 pad 1: /Block Diagram/Auto Zero/AIN_N -> /Block Diagram/Auto Zero/AIN
- R6 pad 2: Net-(R4-Pad2) -> Net-(R6-Pad2)
- R64 pad 1: /Block Diagram/Auto Zero/AIN_P -> Net-(R61-Pad2)
- R64 pad 2: Net-(R64-Pad2) -> /Block Diagram/Analog Channels1/IN
- R7 pad 2: Net-(R4-Pad2) -> Net-(R6-Pad2)
- R8 pad 1: +10V -> Net-(R6-Pad2)
- R8 pad 2: Net-(U1B--) -> Net-(R5-Pad2)
- R9 pad 1: Net-(R4-Pad2) -> Net-(R6-Pad2)
- RN1 pad 3: Net-(R4-Pad2) -> Net-(R6-Pad2)
- RN2 pad 3: Net-(R11-Pad2) -> Net-(R70-Pad2)
- U1 pad 1: Net-(R4-Pad2) -> Net-(R6-Pad2)
- U1 pad 7: Net-(R11-Pad2) -> Net-(R5-Pad2)
- U11 pad 1: /Block Diagram/Analog Channels/OUT_N -> /Block Diagram/Analog Channels1/OUT
- U12 pad 2: /Block Diagram/Auto Zero/AIN_N -> /Block Diagram/Auto Zero/AIN
- U13 pad 1: /Block Diagram/Analog Channels/IN_N -> /Block Diagram/Analog Channels/IN
Routing:
- net /Block Diagram/Auto Zero/AZ_CTR: track 0.00 -> 34.9 mm, vias 0 -> 4
- net Net-(Q8-C): track 0.00 -> 32.1 mm, vias 0 -> 2
- net Net-(Q2-C): track 0.00 -> 32.1 mm, vias 0 -> 2
- net GND: track 0.00 -> 27.1 mm, vias 0 -> 32
- net Net-(Q11-C): track 0.00 -> 25.1 mm, vias 0 -> 3
- net Net-(Q5-C): track 0.00 -> 25.1 mm, vias 0 -> 3
- net Net-(Q3-E): track 0.00 -> 24.7 mm, vias 0 -> 2
- net Net-(Q9-E): track 0.00 -> 24.7 mm, vias 0 -> 2
- net Net-(R6-Pad2): track 0.00 -> 24.4 mm, vias 0 -> 2
- net Net-(R70-Pad2): track 0.00 -> 24.4 mm, vias 0 -> 2
- net +18V: track 0.00 -> 23.4 mm, vias 0 -> 10
- net /Block Diagram/Analog Channels1/OUT: track 0.00 -> 21.8 mm, vias 0 -> 2
- net /Block Diagram/Analog Channels/OUT: track 0.00 -> 21.8 mm, vias 0 -> 2
- net -18V: track 0.00 -> 21.2 mm, vias 0 -> 8
- net Net-(Q4-G): track 0.00 -> 20.7 mm
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Other:
- copper layers 2 -> 4

Commit message: PCB
Parts:
- added D1: DZ2S100X0L, Diode_SMD:D_SOD-523, F.Cu at (186.3, 54.6)
- added H1: MountingHole, MountingHole:MountingHole_3.2mm_M3_DIN965_Pad, F.Cu at (92.0, 44.0)
- added H2: MountingHole, MountingHole:MountingHole_3.2mm_M3_DIN965_Pad, F.Cu at (223.0, 44.0)
- added H3: MountingHole, MountingHole:MountingHole_3.2mm_M3_DIN965_Pad, F.Cu at (92.0, 106.0)
- added H4: MountingHole, MountingHole:MountingHole_3.2mm_M3_DIN965_Pad, F.Cu at (223.0, 106.0)
- added J3: Conn_01x02, TerminalBlock_Phoenix:TerminalBlock_Phoenix_MPT-0,5-2-2.54_1x02_P2.54mm_Horizontal, F.Cu at (190.0, 44.8)
- added Q7: SiS443DN, Package_SO:Vishay_PowerPAK_1212-8_Single, F.Cu at (188.6, 57.7)
- added R12: 0, Resistor_SMD:R_0603_1608Metric, F.Cu at (191.2, 57.4)
- added R13: 100k, Resistor_SMD:R_0603_1608Metric, F.Cu at (185.6, 57.0)
- added R57: 0, Resistor_SMD:R_0603_1608Metric, F.Cu at (169.8, 103.6)
- added R58: 0, Resistor_SMD:R_0603_1608Metric, F.Cu at (161.9, 103.6)
- added TP1: TestPoint, TestPoint:TestPoint_Pad_D2.0mm, F.Cu at (128.0, 71.9)
- added TP10: TestPoint, TestPoint:TestPoint_Pad_D2.0mm, F.Cu at (135.5, 43.3)
- added TP11: TestPoint, TestPoint:TestPoint_Pad_D2.0mm, F.Cu at (157.7, 61.7)
- added TP12: TestPoint, TestPoint:TestPoint_Pad_D2.0mm, F.Cu at (166.8, 43.9)
- added TP13: TestPoint, TestPoint:TestPoint_Pad_D2.0mm, F.Cu at (169.5, 75.2)
- added TP14: TestPoint, TestPoint:TestPoint_Pad_D2.0mm, F.Cu at (175.6, 83.4)
- added TP15: TestPoint, TestPoint:TestPoint_Pad_D2.0mm, F.Cu at (192.9, 71.1)
- added TP16: TestPoint, TestPoint:TestPoint_Pad_D2.0mm, F.Cu at (173.7, 88.3)
- added TP17: TestPoint, TestPoint:TestPoint_Pad_D2.0mm, F.Cu at (173.1, 73.2)
- added TP18: TestPoint, TestPoint:TestPoint_Pad_D2.0mm, F.Cu at (208.2, 85.0)
- added TP19: TestPoint, TestPoint:TestPoint_Pad_D2.0mm, F.Cu at (181.0, 93.6)
- added TP2: TestPoint, TestPoint:TestPoint_Pad_D2.0mm, F.Cu at (126.6, 62.0)
- added TP20: TestPoint, TestPoint:TestPoint_Pad_D2.0mm, F.Cu at (206.4, 75.8)
- added TP21: TestPoint, TestPoint:TestPoint_Pad_D2.0mm, F.Cu at (161.9, 94.6)
- added TP22: TestPoint, TestPoint:TestPoint_Pad_D2.0mm, F.Cu at (158.8, 88.3)
- added TP23: TestPoint, TestPoint:TestPoint_Pad_D2.0mm, F.Cu at (158.9, 70.7)
- added TP24: TestPoint, TestPoint:TestPoint_Pad_D2.0mm, F.Cu at (122.2, 90.8)
- added TP25: TestPoint, TestPoint:TestPoint_Pad_D2.0mm, F.Cu at (211.6, 66.2)
- added TP26: TestPoint, TestPoint:TestPoint_Pad_D2.0mm, F.Cu at (211.8, 73.8)
- added TP27: TestPoint, TestPoint:TestPoint_Pad_D2.0mm, F.Cu at (211.8, 70.0)
- added TP28: TestPoint, TestPoint:TestPoint_Pad_D2.0mm, F.Cu at (156.7, 84.6)
- added TP29: TestPoint, TestPoint:TestPoint_Pad_D2.0mm, F.Cu at (214.3, 64.6)
- added TP3: TestPoint, TestPoint:TestPoint_Pad_D2.0mm, F.Cu at (153.3, 64.9)
- added TP30: TestPoint, TestPoint:TestPoint_Pad_D2.0mm, F.Cu at (214.3, 72.1)
- added TP31: TestPoint, TestPoint:TestPoint_Pad_D2.0mm, F.Cu at (214.3, 68.3)
- added TP32: TestPoint, TestPoint:TestPoint_Pad_D2.0mm, F.Cu at (154.1, 78.5)
- added TP33: TestPoint, TestPoint:TestPoint_Pad_D2.0mm, F.Cu at (128.0, 90.9)
- added TP34: TestPoint, TestPoint:TestPoint_Pad_D2.0mm, F.Cu at (126.6, 81.0)
- added TP35: TestPoint, TestPoint:TestPoint_Pad_D2.0mm, F.Cu at (153.3, 83.9)
- added TP36: TestPoint, TestPoint:TestPoint_Pad_D2.0mm, F.Cu at (150.9, 96.6)
- added TP37: TestPoint, TestPoint:TestPoint_Pad_D2.0mm, F.Cu at (155.7, 87.5)
- added TP4: TestPoint, TestPoint:TestPoint_Pad_D2.0mm, F.Cu at (150.9, 77.6)
- added TP5: TestPoint, TestPoint:TestPoint_Pad_D2.0mm, F.Cu at (155.7, 68.5)
- added TP6: TestPoint, TestPoint:TestPoint_Keystone_5010-5014_Multipurpose, F.Cu at (165.1, 69.5)
- added TP7: TestPoint, TestPoint:TestPoint_Keystone_5010-5014_Multipurpose, F.Cu at (139.8, 78.6)
- added TP8: TestPoint, TestPoint:TestPoint_Pad_D2.0mm, F.Cu at (135.1, 57.1)
- added TP9: TestPoint, TestPoint:TestPoint_Pad_D2.0mm, F.Cu at (156.7, 57.4)
- C11, C13, C33, C39, C42, C9: moved to B.Cu
- R15: renamed from R13; moved to B.Cu
- R21: renamed from R19; moved to B.Cu
- R22: renamed from R20; moved to B.Cu
- R25: renamed from R23; moved to B.Cu
- R28: renamed from R26; moved to B.Cu
- U6: value ADP7142ACPZN -> ADP7142ARDZ; footprint Package_CSP:LFCSP-6-1EP_2x2mm_P0.65mm_EP1x1.6mm -> Package_SO:SOIC-8-1EP_3.9x4.9mm_P1.27mm_EP2.29x3mm
- moved L3 174.6 mm to (141.7, 50.8), turned to 90 degrees
- moved D4 132.3 mm to (137.9, 50.8), turned to 90 degrees
- moved U6 130.5 mm to (130.9, 49.7), turned to -90 degrees
- moved R31 130.4 mm to (133.2, 44.5), turned to 90 degrees
- moved R23 129.1 mm to (130.9, 45.3), turned to 180 degrees
- moved R24 128.6 mm to (130.9, 43.7)
- moved R25 128.4 mm to (130.9, 43.7), turned to 180 degrees
- moved L1 126.1 mm to (187.1, 51.3), turned to 90 degrees
- moved L2 126.0 mm to (149.0, 46.2), turned to 90 degrees
- moved C42 121.1 mm to (175.9, 73.2)
- moved U4 119.8 mm to (148.1, 52.8)
- moved R18 119.4 mm to (137.9, 55.0), turned to -90 degrees
- moved R19 117.5 mm to (139.4, 55.0), turned to 90 degrees
- moved R21 117.0 mm to (139.4, 55.0), turned to -90 degrees
- moved R14 116.3 mm to (142.6, 55.9), turned to 180 degrees
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- renumbered D1 to D2, D2 to D3, D3 to D4, D4 to D5, D5 to D6, J3 to J4, J4 to J5, Q9 to Q10, Q10 to Q11, Q11 to Q12, Q12 to Q13, Q7 to Q8, Q8 to Q9, R12 to R14, R14 to R16, R15 to R17, R16 to R18, R17 to R19, R18 to R20, R21 to R23, R22 to R24, R24 to R26, R25 to R27, R27 to R29, R28 to R30, R29 to R31, R30 to R32, R31 to R33, R32 to R34, R33 to R35, R34 to R36, R35 to R37, R36 to R38, R37 to R39, R38 to R40, R39 to R41, R40 to R42, R41 to R43, R42 to R44, R43 to R45, R44 to R46, R45 to R47, R46 to R48, R47 to R49, R48 to R50, R49 to R51, R50 to R52, R51 to R53, R52 to R54, R53 to R55, R54 to R56, R55 to R59, R56 to R60, R57 to R61, R58 to R62, R59 to R63, R60 to R64, R61 to R65, R62 to R66, R63 to R67, R64 to R68, R65 to R69, R66 to R70, R67 to R71, R68 to R72, R69 to R73, R70 to R74, R71 to R75, R72 to R76, R73 to R77, R74 to R78, U18 to U17, U17 to U18
Connections:
- C16 pad 1: Net-(D3-K) (its old number) -> Net-(D4-K)
- C17 pad 1: GND -> Net-(D3-A)
- C19 pad 1: Net-(D3-K) (its old number) -> Net-(D4-K)
- C20 pad 2: GND -> Net-(D3-A)
- C21 pad 2: GND -> Net-(D3-A)
- D3 pad 2: GND -> Net-(D3-A)
- D4 pad 1: Net-(D3-K) (its old number) -> Net-(D4-K)
- R17 pad 1: GND -> Net-(D3-A)
- R18 pad 1: Net-(D3-K) (its old number) -> Net-(D4-K)
- R23 pad 1: Net-(U6-VOUT) -> Net-(R23-Pad1)
- R23 pad 2: Net-(U6-ADJ) -> Net-(U6-SENSE/ADJ)
- R24 pad 1: Net-(U6-ADJ) -> Net-(U6-SENSE/ADJ)
- R31 pad 1: Net-(U6-VOUT) -> Net-(R23-Pad1)
- U14 pad 5: Net-(U14-Pad5) -> -7V
- U16 pad 8: Net-(U14-Pad5) -> -7V
- U24 pad 3: +18V -> Net-(U24-HEATER+)
- U24 pad 5: -18V -> Net-(U24-HEATER-)
- U6 pad 1: Net-(U6-VOUT) -> Net-(R23-Pad1)
- U6 pad 2: Net-(U6-ADJ) -> Net-(R23-Pad1)
- U6 pad 3: GND -> Net-(U6-SENSE/ADJ)
- U6 pad 4: Net-(D3-K) (its old number) -> GND
- U6 pad 5: unconnected-(U6-SS-Pad5) -> Net-(D4-K)
- U6 pad 6: Net-(D3-K) (its old number) -> unconnected-(U6-SS-Pad6)
- U6 pad 7: GND -> Net-(D4-K)
- U7 pad 3: GND -> Net-(D3-A)
- U7 pad 6: GND -> Net-(D3-A)
- U7 pad 7: GND -> Net-(D3-A)
- U8 pad 3: GND -> Net-(D3-A)
- U8 pad 6: GND -> Net-(D3-A)
- U8 pad 7: GND -> Net-(D3-A)
Routing:
- net +18V: track 23.4 -> 330.3 mm, vias 10 -> 17
- net +3.3V: track 9.61 -> 260.7 mm, vias 4 -> 11
- net -18V: track 21.2 -> 241.2 mm, vias 8 -> 14
- net /Block Diagram/Auto Zero/AZ_CTR: track 34.9 -> 150.3 mm
- net -14V: track 0.00 -> 94.7 mm, vias 0 -> 4
- net /Block Diagram/Gain/GAIN_x100: track 0.00 -> 90.7 mm, vias 0 -> 1
- net /Block Diagram/Gain/GAIN_x10: track 0.00 -> 79.4 mm, vias 0 -> 1
- net /Block Diagram/ADC/AD_COMP: track 0.00 -> 55.0 mm, vias 0 -> 2
- net /Block Diagram/ADC/FGPA_AD_ID: track 0.00 -> 52.2 mm, vias 0 -> 2
- net /Block Diagram/ADC/FPGA_SW_VRH: track 0.00 -> 51.9 mm, vias 0 -> 2
- net /Block Diagram/ADC/FGPA_AD_IRN: track 0.00 -> 51.8 mm, vias 0 -> 2
- net /Block Diagram/ADC/FGPA_AD_IRP: track 0.00 -> 51.7 mm, vias 0 -> 2
- net /Block Diagram/ADC/FGPA_AD_IIN: track 0.00 -> 51.4 mm, vias 0 -> 2
- net +10V: track 0.83 -> 49.4 mm, vias 1 -> 4
- net GND: track 27.1 -> 73.9 mm, vias 32 -> 80
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- added copper zone on B.Cu, net GND
- added copper zone on F.Cu, net GND
- added copper zone on In1.Cu, net GND
Other:
- board outline added: 139 x 70 mm

Commit message: Schematic
Parts:
- moved TP26 4.17 mm to (212.1, 69.6)
- moved TP27 4.17 mm to (212.1, 65.8)
- moved J5 4.17 mm to (220.2, 56.8)
- moved TP25 4.17 mm to (212.0, 62.0)
- moved TP29 4.17 mm to (214.7, 60.5)
- moved TP30 4.17 mm to (214.7, 68.0)
- moved TP31 4.17 mm to (214.7, 64.2)
- moved J4 2.42 mm to (220.2, 79.6)
Connections:
- J5 pad 10: /Block Diagram/ADC/AD_COMP -> /Block Diagram/ADC/FGPA_AD_IIN
- J5 pad 5: /Block Diagram/ADC/FGPA_AD_IIN -> /Block Diagram/ADC/FGPA_AD_ID
- J5 pad 6: /Block Diagram/ADC/FGPA_AD_ID -> /Block Diagram/ADC/AD_COMP
- TP25 pad 1: /Block Diagram/ADC/FGPA_AD_IIN -> /Block Diagram/ADC/FGPA_AD_ID
- TP29 pad 1: /Block Diagram/ADC/FGPA_AD_ID -> /Block Diagram/ADC/AD_COMP
- TP30 pad 1: /Block Diagram/ADC/AD_COMP -> /Block Diagram/ADC/FGPA_AD_IIN
Routing:
- net /Block Diagram/Gain/GAIN_x100: track 90.7 -> 4.62 mm
- net /Block Diagram/Gain/GAIN_x10: track 79.4 -> 3.83 mm
- net /Block Diagram/Auto Zero/AZ_CTR: track 150.3 -> 162.4 mm
- net /Block Diagram/ADC/AD_COMP: track 55.0 -> 50.9 mm
- net Net-(U15-Pad5): track 16.3 -> 13.8 mm
- net /Block Diagram/ADC/FGPA_AD_ID: track 52.2 -> 50.8 mm
- net /Block Diagram/ADC/FGPA_AD_IRP: track 51.7 -> 50.8 mm
- net /Block Diagram/ADC/FGPA_AD_IIN: track 51.4 -> 52.1 mm
- net /Block Diagram/ADC/FGPA_AD_IRN: track 51.8 -> 51.3 mm
