File: Hardware/MADC_ARTY/PMOD.kicad_sch (KiCad schematic)
At the start: 11 parts, among them J4 71764-0012, J5 71764-0012

Commit message: PCB and schematic
Parts:
- added R70: 0, Resistor_SMD:R_0603_1608Metric, symbol Device:R
- TP18, TP19, TP20, TP21, TP22, TP23, TP24, TP25, TP26: now left out of the parts list
Connections:
- net +3.3VP: now reaches J5.1 (Pin_1)
- net +3.3VP: now also J4.1 (Pin_1), J4.2 (Pin_2), J5.2 (Pin_2), R70.2
- new net +3.3V: R70.1
- no-connect marks 11 -> 7
Other:
- moved on the sheet: J4, J5, TP18, TP19, TP20, TP21, TP22, TP23, TP24, TP25, TP26

Commit message: BOM
Parts:
- renumbered R70 to R64, TP18 to TP21, TP19 to TP22, TP20 to TP23, TP21 to TP24, TP22 to TP25, TP23 to TP26, TP24 to TP27, TP25 to TP28, TP26 to TP29
Changed lines of the file:
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@@
 		(dnp no)
 		(fields_autoplaced yes)
-		(property "Reference" "TP23"
+		(property "Reference" "TP26"
 			(at 218.44 94.4879 0)
 			(effects
@@
 			(project "MADC_ARTY"
 				(path "/eadab778-ea7c-433e-b0bd-0d0c238907e0/37dfacfc-f3f5-4a09-9e7e-ab0b8ea302f6/5d4b0f99-b739-4f3c-9f1e-19d2c8b0b121"
-					(reference "TP23")
+					(reference "TP26")
 					(unit 1)
 				)
@@
 		(dnp no)
 		(fields_autoplaced yes)
-		(property "Reference" "TP24"
+		(property "Reference" "TP27"
 			(at 218.44 118.8721 0)
 			(effects
@@
 			(project "MADC_ARTY"
 				(path "/eadab778-ea7c-433e-b0bd-0d0c238907e0/37dfacfc-f3f5-4a09-9e7e-ab0b8ea302f6/5d4b0f99-b739-4f3c-9f1e-19d2c8b0b121"
-					(reference "TP24")
+					(reference "TP27")
 					(unit 1)
 				)
@@
 		(dnp no)
 		(fields_autoplaced yes)
-		(property "Reference" "TP18"
+		(property "Reference" "TP21"
 			(at 57.15 97.0279 0)
 			(effects
@@
 			(project "MADC_ARTY"
 				(path "/eadab778-ea7c-433e-b0bd-0d0c238907e0/37dfacfc-f3f5-4a09-9e7e-ab0b8ea302f6/5d4b0f99-b739-4f3c-9f1e-19d2c8b0b121"
-					(reference "TP18")
+					(reference "TP21")
 					(unit 1)
 				)
@@
 		(dnp no)
 		(fields_autoplaced yes)
-		(property "Reference" "#PWR103"
+		(property "Reference" "#PWR0134"
 			(at 205.74 100.33 0)
 			(effects
@@
 			(project "MADC_ARTY"
 				(path "/eadab778-ea7c-433e-b0bd-0d0c238907e0/37dfacfc-f3f5-4a09-9e7e-ab0b8ea302f6/5d4b0f99-b739-4f3c-9f1e-19d2c8b0b121"
-					(reference "#PWR103")
+					(reference "#PWR0134")
 					(unit 1)
 				)
@@
 		(dnp no)
 		(fields_autoplaced yes)
-		(property "Reference" "TP21"
+		(property "Reference" "TP24"
 			(at 165.1 94.4879 0)
 			(effects
@@
 			(project "MADC_ARTY"
 				(path "/eadab778-ea7c-433e-b0bd-0d0c238907e0/37dfacfc-f3f5-4a09-9e7e-ab0b8ea302f6/5d4b0f99-b739-4f3c-9f1e-19d2c8b0b121"
-					(reference "TP21")
+					(reference "TP24")
 					(unit 1)
 				)
@@
 		(dnp no)
 		(fields_autoplaced yes)
-		(property "Reference" "TP19"
+		(property "Reference" "TP22"
 			(at 152.4 94.4879 0)
 			(effects
@@
 			(project "MADC_ARTY"
 				(path "/eadab778-ea7c-433e-b0bd-0d0c238907e0/37dfacfc-f3f5-4a09-9e7e-ab0b8ea302f6/5d4b0f99-b739-4f3c-9f1e-19d2c8b0b121"
-					(reference "TP19")
+					(reference "TP22")
 					(unit 1)
 				)
@@
 		(dnp no)
 		(fields_autoplaced yes)
-		(property "Reference" "#PWR0140"
+		(property "Reference" "#PWR0130"
 			(at 187.96 93.98 0)
 			(effects
@@
 			(project ""
 				(path "/eadab778-ea7c-433e-b0bd-0d0c238907e0/37dfacfc-f3f5-4a09-9e7e-ab0b8ea302f6/5d4b0f99-b739-4f3c-9f1e-19d2c8b0b121"
-					(reference "#PWR0140")
+					(reference "#PWR0130")
 					(unit 1)
 				)
@@
 		(dnp no)
 		(fields_autoplaced yes)
-		(property "Reference" "#PWR100"
+		(property "Reference" "#PWR0126"
 			(at 74.93 100.33 0)
 			(effects
@@
 			(project "MADC_ARTY"
 				(path "/eadab778-ea7c-433e-b0bd-0d0c238907e0/37dfacfc-f3f5-4a09-9e7e-ab0b8ea302f6/5d4b0f99-b739-4f3c-9f1e-19d2c8b0b121"
-					(reference "#PWR100")
+					(reference "#PWR0126")
 					(unit 1)
 				)
@@
 		(dnp no)
 		(fields_autoplaced yes)
-		(property "Reference" "#FLG09"
+		(property "Reference" "#FLG014"
 			(at 25.4 187.325 0)
 			(effects
@@
 			(project ""
 				(path "/eadab778-ea7c-433e-b0bd-0d0c238907e0/37dfacfc-f3f5-4a09-9e7e-ab0b8ea302f6/5d4b0f99-b739-4f3c-9f1e-19d2c8b0b121"
-					(reference "#FLG09")
+					(reference "#FLG014")
 					(unit 1)
 				)
@@
 		(dnp no)
 		(fields_autoplaced yes)
-		(property "Reference" "#PWR102"
+		(property "Reference" "#PWR0131"
 			(at 180.34 100.33 0)
 			(effects
@@
 			(project "MADC_ARTY"
 				(path "/eadab778-ea7c-433e-b0bd-0d0c238907e0/37dfacfc-f3f5-4a09-9e7e-ab0b8ea302f6/5d4b0f99-b739-4f3c-9f1e-19d2c8b0b121"
-					(reference "#PWR102")
+					(reference "#PWR0131")
 					(unit 1)
 				)
@@
 		(dnp no)
 		(fields_autoplaced yes)
-		(property "Reference" "#PWR101"
+		(property "Reference" "#PWR0128"
 			(at 100.33 100.33 0)
 			(effects
@@
 			(project "MADC_ARTY"
 				(path "/eadab778-ea7c-433e-b0bd-0d0c238907e0/37dfacfc-f3f5-4a09-9e7e-ab0b8ea302f6/5d4b0f99-b739-4f3c-9f1e-19d2c8b0b121"
-					(reference "#PWR101")
+					(reference "#PWR0128")
 					(unit 1)
 				)
@@
 		(dnp no)
 		(fields_autoplaced yes)
-		(property "Reference" "TP20"
+		(property "Reference" "TP23"
 			(at 152.4 116.3319 0)
 			(effects
@@
 			(project "MADC_ARTY"
 				(path "/eadab778-ea7c-433e-b0bd-0d0c238907e0/37dfacfc-f3f5-4a09-9e7e-ab0b8ea302f6/5d4b0f99-b739-4f3c-9f1e-19d2c8b0b121"
-					(reference "TP20")
+					(reference "TP23")
 					(unit 1)
 				)
@@
 		(dnp no)
 		(fields_autoplaced yes)
-		(property "Reference" "#PWR0155"
+		(property "Reference" "#PWR0124"
 			(at 29.21 186.69 0)
 			(effects
@@
 			(project "MADC_ARTY"
 				(path "/eadab778-ea7c-433e-b0bd-0d0c238907e0/37dfacfc-f3f5-4a09-9e7e-ab0b8ea302f6/5d4b0f99-b739-4f3c-9f1e-19d2c8b0b121"
-					(reference "#PWR0155")
+					(reference "#PWR0124")
 					(unit 1)
 				)
@@
 		(dnp no)
 		(fields_autoplaced yes)
-		(property "Reference" "R70"
+		(property "Reference" "R64"
 			(at 193.04 82.55 90)
 			(effects
@@
 			(project ""
 				(path "/eadab778-ea7c-433e-b0bd-0d0c238907e0/37dfacfc-f3f5-4a09-9e7e-ab0b8ea302f6/5d4b0f99-b739-4f3c-9f1e-19d2c8b0b121"
-					(reference "R70")
+					(reference "R64")
 					(unit 1)
 				)
@@
 		(dnp no)
 		(fields_autoplaced yes)
-		(property "Reference" "TP25"
+		(property "Reference" "TP28"
 			(at 231.14 94.4879 0)
 			(effects
@@
 			(project "MADC_ARTY"
 				(path "/eadab778-ea7c-433e-b0bd-0d0c238907e0/37dfacfc-f3f5-4a09-9e7e-ab0b8ea302f6/5d4b0f99-b739-4f3c-9f1e-19d2c8b0b121"
-					(reference "TP25")
+					(reference "TP28")
 					(unit 1)
 				)
@@
 		(dnp no)
 		(fields_autoplaced yes)
-		(property "Reference" "TP22"
+		(property "Reference" "TP25"
 			(at 165.1 116.3319 0)
 			(effects
@@
 			(project "MADC_ARTY"
 				(path "/eadab778-ea7c-433e-b0bd-0d0c238907e0/37dfacfc-f3f5-4a09-9e7e-ab0b8ea302f6/5d4b0f99-b739-4f3c-9f1e-19d2c8b0b121"
-					(reference "TP22")
+					(reference "TP25")
 					(unit 1)
 				)
@@
 		(dnp no)
 		(fields_autoplaced yes)
-		(property "Reference" "#PWR0153"
+		(property "Reference" "#PWR0125"
 			(at 82.55 93.98 0)
 			(effects
@@
 			(project "MADC_ARTY"
 				(path "/eadab778-ea7c-433e-b0bd-0d0c238907e0/37dfacfc-f3f5-4a09-9e7e-ab0b8ea302f6/5d4b0f99-b739-4f3c-9f1e-19d2c8b0b121"
-					(reference "#PWR0153")
+					(reference "#PWR0125")
 					(unit 1)
 				)
@@
 		(dnp no)
 		(fields_autoplaced yes)
-		(property "Reference" "#PWR0154"
+		(property "Reference" "#PWR0127"
 			(at 92.71 101.6 0)
 			(effects
@@
 			(project "MADC_ARTY"
 				(path "/eadab778-ea7c-433e-b0bd-0d0c238907e0/37dfacfc-f3f5-4a09-9e7e-ab0b8ea302f6/5d4b0f99-b739-4f3c-9f1e-19d2c8b0b121"
-					(reference "#PWR0154")
+					(reference "#PWR0127")
 					(unit 1)
 				)
@@
 		(dnp no)
 		(fields_autoplaced yes)
-		(property "Reference" "#PWR0141"
+		(property "Reference" "#PWR0133"
 			(at 198.12 101.6 0)
 			(effects
@@
 			(project "MADC_ARTY"
 				(path "/eadab778-ea7c-433e-b0bd-0d0c238907e0/37dfacfc-f3f5-4a09-9e7e-ab0b8ea302f6/5d4b0f99-b739-4f3c-9f1e-19d2c8b0b121"
-					(reference "#PWR0141")
+					(reference "#PWR0133")
 					(unit 1)
 				)
@@
 		(dnp no)
 		(fields_autoplaced yes)
-		(property "Reference" "#PWR0142"
+		(property "Reference" "#PWR0129"
 			(at 190.5 88.9 0)
 			(effects
@@
 			(project ""
 				(path "/eadab778-ea7c-433e-b0bd-0d0c238907e0/37dfacfc-f3f5-4a09-9e7e-ab0b8ea302f6/5d4b0f99-b739-4f3c-9f1e-19d2c8b0b121"
-					(reference "#PWR0142")
+					(reference "#PWR0129")
 					(unit 1)
 				)
@@
 		(dnp no)
 		(fields_autoplaced yes)
-		(property "Reference" "#PWR0143"
+		(property "Reference" "#PWR0132"
 			(at 198.12 92.71 0)
 			(effects
@@
 			(project "MADC_ARTY"
 				(path "/eadab778-ea7c-433e-b0bd-0d0c238907e0/37dfacfc-f3f5-4a09-9e7e-ab0b8ea302f6/5d4b0f99-b739-4f3c-9f1e-19d2c8b0b121"
-					(reference "#PWR0143")
+					(reference "#PWR0132")
 					(unit 1)
 				)
@@
 		(dnp no)
 		(fields_autoplaced yes)
-		(property "Reference" "TP26"
+		(property "Reference" "TP29"
 			(at 231.14 118.8721 0)
 			(effects
@@
 			(project "MADC_ARTY"
 				(path "/eadab778-ea7c-433e-b0bd-0d0c238907e0/37dfacfc-f3f5-4a09-9e7e-ab0b8ea302f6/5d4b0f99-b739-4f3c-9f1e-19d2c8b0b121"
-					(reference "TP26")
-					(unit 1)
-				)
+					(reference "TP29")
+					(unit 1)
+				)
